File: Python_STM32/docs/DSP board HW/Main Board/MCU.kicad_sch (KiCad schematic)
At the start: 2 parts, among them U7 STM32H725ZGTx

Commit message: Board design largely done
Parts:
- removed U7: STM32H725ZGTx, Package_QFP:LQFP-144_20x20mm_P0.5mm, symbol MCU_ST_STM32H7:STM32H725ZGTx
- added C100, C102, C90, C91, C92, C96, C97, C98, C99: 100nF, symbol Device:C
- added C101, C95: 4.7uF, symbol Device:C
- added C103: 1uF, symbol Device:C
- added C2: 100nF, symbol Device:C_Small
- added C93, C94: 15pF, symbol Device:C
- added L2: 2.2uH, symbol Device:L
- added R18: 10K, symbol Device:R
- added U7: STM32H725RGVx, symbol MCU_ST_STM32H7:STM32H725RGVx
- added Y1: 24.576MHz, symbol Device:Crystal
Connections:
- net 3V45_D: now also C100.1, C101.1, C96.1, C97.1, C98.1, C99.1, U7.1 (VBAT), U7.22 (VDD), U7.35 (VDD), U7.51 (VDD), U7.6 (VDDSMPS), U7.68 (VDD), U7.9 (VDD)
- net BATT_SENSE: now also U7.27 (PC4)
- net BT1: now also U7.36 (PB12)
- net BT2: now also U7.39 (PB15)
- net CODEC_SHDNZ: now also R18.1, U7.40 (PC6)
- net GND: now also C100.2, C101.2, C102.2, C103.2, C2.1, C90.2, C91.2, C92.2, C93.2, C94.2, C95.2, C96.2, C97.2, C98.2, C99.2, R18.2, U7.15 (VSSA), U7.21 (VSS), U7.34 (VSS), U7.4 (VSSSMPS), U7.50 (VSS), U7.67 (VSS), U7.69 (VSS), U7.8 (VSS)
- net I2C1_SCL: now also U7.64 (PB8)
- net I2C1_SDA: now also U7.65 (PB9)
- net LED: now also U7.57 (PD2)
- net MCO1: now also U7.43 (PA8)
- net MCU_VDDA: now also C102.1, C103.1, U7.16 (VDDA)
- net OTG_FS_DM: now also U7.46 (PA11)
- net OTG_FS_DP: now also U7.47 (PA12)
- net Pot2: now also U7.14 (PC1)
- net Pot3: now also U7.28 (PC5)
- net SWCLK: now also U7.52 (PA14(JTCK)
- net SWDIO: now also U7.48 (PA13(JTMS)
- net USART3_CTS: now also U7.37 (PB13)
- net USART3_RTS: now also U7.38 (PB14)
- net USART3_RX: now also U7.55 (PC11)
- net USART3_TX: now also U7.54 (PC10)
- net at R14.2: now also U7.63 (BOOT0)
- new net: C94.1, U7.11 (PH1), Y1.1
- new net: C93.1, U7.10 (PH0), Y1.2
- new net: C90.1, U7.33 (VCAP)
- new net: C91.1, U7.49 (VCAP)
- new net: L2.2, U7.5 (VLXSMPS)
- new net: C92.1, U7.66 (VCAP)
- new net: C95.1, L2.1, U7.7 (VFBSMPS)
- new net DAC_XSMT: U7.42 (PC9)
- new net I2S1_CK: U7.24 (PA5)
- new net I2S1_SDO: U7.26 (PA7)
- new net I2S1_WS: U7.23 (PA4)
- new net NRST: C2.2, U7.12 (NRST)
- new net SAI4_FS_B: U7.13 (PC0)
- new net SAI4_SCK_B: U7.19 (PA2)
- new net SAI4_SD_B: U7.17 (PA0)
- new net SWO: U7.58 (PB3(JTDO)
Other:
- note added: "Decoupling - one 100nF per VDD pin + 4.7uF bulk, place at U7. VDDA pair at pin 16."
- note added: "HSE 24.576 MHz - integer-N PLL3 for 48k family"
- note added: "SMPS direct (AN5419): 2.2uH VLX->VFB, 4.7uF at VFB"

Commit message: Update DSP board HW docs
Parts:
- added TP1: MC01, symbol Connector:TestPoint
- added TP10: (no value), symbol Connector:TestPoint
Connections:
- net CODEC_SHDNZ: now also TP10.1
- net MCO1: no longer names the net of U7.43 (PA8)
- net MCO1: now also TP1.1
