File: Python_STM32/docs/DSP board HW/Main Board/Main Board.kicad_sch (KiCad schematic)
At the start: 62 parts, among them J1 Bridge Pickup, J2 Neck Pickup, J3 Battery, J4 Output Jack, U1 TPS7A2033PDBVR, U2 TPS63020DSJR, U3 XLV320ADC5140IRTWR, U4 XLV320ADC5140IRTWR, U6 PCM5102, U8 TP4054

Commit message: Board design largely done
Parts:
- added C37: 1uF, symbol Device:C_Small
- added C38: 100nF, symbol Device:C_Small
- added D1: LED, symbol Device:LED
- added J5: Debug Connector, symbol Connector_Generic:Conn_02x05_Odd_Even
- added R15: R, symbol Device:R
- FB1: value FerriteBead -> 600
Connections:
- net 3V45_D: now also J5.1 (Pin_1)
- net GND: now also C37.1, C38.1, J5.3 (Pin_3), J5.5 (Pin_5), J5.9 (Pin_9), R15.2
- net MCU_VDDA: now also C37.2, C38.2
- net at C25.1: now also U4.13 (IN4M_GPO4)
- net PD15 renamed DAC_XSMT
- net SAI1_FS_A renamed SAI4_FS_B
- net SAI1_FS_B renamed I2S1_WS
- net SAI1_SCK_A renamed SAI4_SCK_B
- net SAI1_SCK_B renamed I2S1_CK
- net SAI1_SD_A renamed SAI4_SD_B
- net SAI1_SD_B renamed I2S1_SDO
- new net: D1.1 (K), R15.1
- new net LED: D1.2 (A)
- new net NRST: J5.10 (Pin_10)
- new net SWCLK: J5.4 (Pin_4)
- new net SWDIO: J5.2 (Pin_2)
- new net SWO: J5.6 (Pin_6)
Other:
- moved on the sheet: C25, FB1

Commit message: Update DSP board HW docs
Parts:
- added TP11, TP2, TP3, TP4, TP5, TP6, TP7, TP8, TP9: (no value), symbol Connector:TestPoint
Connections:
- net 3V3_A: now also TP3.1
- net 3V45_D: now also TP2.1
- net I2S1_CK: now also TP9.1
- net I2S1_SDO: now also TP8.1
- net I2S1_WS: now also TP7.1
- net SAI4_FS_B: now also TP6.1
- net SAI4_SCK_B: now also TP5.1
- net SAI4_SD_B: now also TP4.1
- net at C35.1, J1.1 (Pin_1), U3.5 (MICBIAS): now also TP11.1
