File: Onboard DSP Board HW/Main Board/Main Board.kicad_pcb (KiCad board)
At the start: 4 copper layers, 25 x 55.8 mm, 21 parts, among them J1 Pickup1, J2 Pickup 2, J3 Vol Pot & Sw, J4 Battery, J5 Dual Pot Board, J6 Output Jack, U1 TL972, U2 MCP73811T-420I-OT

Commit message: WIP
Parts:
- removed A1: Device_Audio_Electrosmith_Daisy_Seed_Rev4, Device_Audio_Electrosmith_Daisy_Seed:Device_Audio_Electrosmith_Daisy_Seed
- removed D1: D, Diode_SMD:D_0603_1608Metric
- removed J1: Pickup1, Connector_PinHeader_1.00mm:PinHeader_1x02_P1.00mm_Vertical
- removed J2: Pickup 2, Connector_PinHeader_1.00mm:PinHeader_1x02_P1.00mm_Vertical
- removed J5: Dual Pot Board, Connector_PinHeader_1.00mm:PinHeader_1x04_P1.00mm_Vertical
- removed J6: Output Jack, Connector_PinHeader_1.00mm:PinHeader_1x03_P1.00mm_Vertical
- added C10: 2.2uF, Capacitor_SMD:C_0402_1005Metric, F.Cu at (130.2, 56.8)
- added C100: 100nF, Capacitor_SMD:C_0402_1005Metric, F.Cu at (156.0, 52.7)
- added C101: 4.7uF, Capacitor_SMD:C_0402_1005Metric, F.Cu at (159.2, 63.5)
- added C102: 100nF, Capacitor_SMD:C_0402_1005Metric, F.Cu at (152.8, 66.2)
- added C103: 1uF, Capacitor_SMD:C_0402_1005Metric, F.Cu at (149.0, 66.0)
- added C11: 2.2uF, Capacitor_SMD:C_0402_1005Metric, F.Cu at (140.5, 55.2)
- added C12: .1uF, Capacitor_SMD:C_0402_1005Metric, F.Cu at (130.2, 58.8)
- added C13: .1uF, Capacitor_SMD:C_0402_1005Metric, F.Cu at (132.8, 53.0)
- added C14: .1uF, Capacitor_SMD:C_0402_1005Metric, F.Cu at (140.5, 54.0)
- added C15: 4.7uF, Capacitor_SMD:C_0402_1005Metric, F.Cu at (119.5, 56.8)
- added C16: 4.7uF, Capacitor_SMD:C_0402_1005Metric, F.Cu at (117.8, 56.8)
- added C17: 4.7uF, Capacitor_SMD:C_0402_1005Metric, F.Cu at (116.2, 56.8)
- added C18: 4.7uF, Capacitor_SMD:C_1206_3216Metric, F.Cu at (107.8, 52.8)
- added C19: 4.7uF, Capacitor_SMD:C_1206_3216Metric, F.Cu at (105.0, 52.8)
- added C20: 4.7uF, Capacitor_SMD:C_1206_3216Metric, F.Cu at (102.2, 52.8)
- added C21: 4.7uF, Capacitor_SMD:C_1206_3216Metric, F.Cu at (99.2, 52.7)
- added C22: 4.7uF, Capacitor_SMD:C_0402_1005Metric, F.Cu at (106.0, 57.0)
- added C23: 4.7uF, Capacitor_SMD:C_0402_1005Metric, F.Cu at (185.1, 57.2)
- added C24: 4.7uF, Capacitor_SMD:C_0402_1005Metric, F.Cu at (104.2, 57.0)
- added C25: 4.7uF, Capacitor_SMD:C_0402_1005Metric, F.Cu at (100.8, 57.0)
- added C26: 4.7uF, Capacitor_SMD:C_0402_1005Metric, F.Cu at (102.5, 57.0)
- added C28: 1uF, Capacitor_SMD:C_0402_1005Metric, F.Cu at (119.8, 63.8)
- added C29: 1uF, Capacitor_SMD:C_0402_1005Metric, F.Cu at (106.2, 64.0)
- added C30: 4.7uF, Capacitor_SMD:C_0402_1005Metric, F.Cu at (178.6, 56.8)
- added C31: 1uF, Capacitor_SMD:C_0402_1005Metric, F.Cu at (121.8, 61.8)
- added C32: 1uF, Capacitor_SMD:C_0402_1005Metric, F.Cu at (121.8, 60.8)
- added C33: 1uF, Capacitor_SMD:C_0402_1005Metric, F.Cu at (108.0, 62.5)
- added C34: 1uF, Capacitor_SMD:C_0402_1005Metric, F.Cu at (108.2, 61.2)
- added C35: 1uF, Capacitor_SMD:C_0402_1005Metric, F.Cu at (121.8, 59.8)
- added C36: 1uF, Capacitor_SMD:C_0402_1005Metric, F.Cu at (108.2, 60.0)
- added C37: 1uF, Capacitor_SMD:C_0402_1005Metric, F.Cu at (159.5, 50.2)
- added C38: 100nF, Capacitor_SMD:C_0402_1005Metric, F.Cu at (159.5, 51.5)
- added C4: 4.7uF, Capacitor_SMD:C_1206_3216Metric, F.Cu at (122.3, 52.8)
- added C5: 4.7uF, Capacitor_SMD:C_1206_3216Metric, F.Cu at (119.5, 52.8)
- added C6: 4.7uF, Capacitor_SMD:C_1206_3216Metric, F.Cu at (116.8, 52.8)
- added C7: 2.2uF, Capacitor_SMD:C_0402_1005Metric, F.Cu at (130.2, 54.8)
- added C8: 4.7uF, Capacitor_SMD:C_1206_3216Metric, F.Cu at (114.0, 52.8)
- added C9: 4.7uF, Capacitor_SMD:C_0402_1005Metric, F.Cu at (114.8, 56.8)
- added C90: 100nF, Capacitor_SMD:C_0402_1005Metric, F.Cu at (151.6, 52.7)
- added C91: 100nF, Capacitor_SMD:C_0402_1005Metric, F.Cu at (148.3, 61.5)
- added C92: 100nF, Capacitor_SMD:C_0402_1005Metric, F.Cu at (157.2, 64.5)
- added C93: 15pF, Capacitor_SMD:C_0402_1005Metric, F.Cu at (163.3, 59.4)
- added C94: 15pF, Capacitor_SMD:C_0402_1005Metric, F.Cu at (163.0, 54.7)
- added C95: 4.7uF, Capacitor_SMD:C_0402_1005Metric, F.Cu at (164.1, 61.3)
- added C96: 100nF, Capacitor_SMD:C_0402_1005Metric, F.Cu at (160.6, 59.5)
- added C97: 100nF, Capacitor_SMD:C_0402_1005Metric, F.Cu at (144.0, 64.2)
- added C98: 100nF, Capacitor_SMD:C_0402_1005Metric, F.Cu at (149.5, 62.5)
- added C99: 100nF, Capacitor_SMD:C_0402_1005Metric, F.Cu at (149.0, 55.2)
- added D2: BAS316, Diode_SMD:D_SOD-323, F.Cu at (126.0, 52.6)
- added L1: 1.5uH, Inductor_SMD:L_Sunlord_SWPA4030S, F.Cu at (181.6, 68.3)
- added L2: 2.2uH, Inductor_SMD:L_Sunlord_SWPA252012S, F.Cu at (162.1, 61.5)
- added R10: 100K, Resistor_SMD:R_0402_1005Metric, F.Cu at (177.8, 63.3)
- added R11: 1M, Resistor_SMD:R_0402_1005Metric, F.Cu at (185.3, 62.3)
- added R12: 1M, Resistor_SMD:R_0402_1005Metric, F.Cu at (153.3, 52.2)
- added R13: 1M, Resistor_SMD:R_0402_1005Metric, F.Cu at (154.8, 52.7)
- added R14: 10K, Resistor_SMD:R_0402_1005Metric, F.Cu at (155.1, 64.2)
- added R15: R, Resistor_SMD:R_0402_1005Metric, F.Cu at (169.7, 74.0)
- added R17: 30k, Resistor_SMD:R_0402_1005Metric, F.Cu at (178.6, 58.8)
- added R18: 10K, Resistor_SMD:R_0402_1005Metric, F.Cu at (148.3, 57.3)
- added RV1: 10K, Resistor_SMD:R_0402_1005Metric, F.Cu at (135.2, 67.2)
- added RV2: 10K, Resistor_SMD:R_0402_1005Metric, F.Cu at (146.8, 67.2)
- added U3: XLV320ADC5140IRTWR, Package_DFN_QFN:HVQFN-24-1EP_4x4mm_P0.5mm_EP2.1x2.1mm, F.Cu at (117.5, 60.5)
- added U4: XLV320ADC5140IRTWR, Package_DFN_QFN:HVQFN-24-1EP_4x4mm_P0.5mm_EP2.1x2.1mm, F.Cu at (104.0, 60.8)
- added U6: PCM5102, Package_SO:TSSOP-20_4.4x6.5mm_P0.65mm, F.Cu at (135.2, 57.0)
- added U7: STM32H725RGVx, Package_DFN_QFN:QFN-68-1EP_8x8mm_P0.4mm_EP6.4x6.4mm, F.Cu at (154.6, 58.5)
- added U8: TP4054, Package_TO_SOT_SMD:SOT-23-5, F.Cu at (182.1, 57.8)
- added Y1: 24.576MHz, Crystal:Crystal_SMD_3225-4Pin_3.2x2.5mm, F.Cu at (162.3, 57.0)
- C1: value 4.7u -> C; footprint Capacitor_SMD:C_0201_0603Metric -> Capacitor_SMD:C_0402_1005Metric
- C2: value 4.7u -> 100nF; footprint Capacitor_SMD:C_0201_0603Metric -> Capacitor_SMD:C_0402_1005Metric
- J3: value Vol Pot & Sw -> Battery; footprint Connector_PinHeader_1.00mm:PinHeader_1x05_P1.00mm_Vertical -> Connector_JST:JST_PH_S2B-PH-K_1x02_P2.00mm_Horizontal
- J4: value Battery -> Output Jack; footprint Connector_PinHeader_1.00mm:PinHeader_1x02_P1.00mm_Vertical -> Connector_PinHeader_2.54mm:PinHeader_1x03_P2.54mm_Vertical
- R1, R2, R5, R6: value 2M -> R; footprint Resistor_SMD:R_0603_1608Metric -> Resistor_SMD:R_0402_1005Metric
- R3, R4: value R_US -> R; footprint Resistor_SMD:R_0603_1608Metric -> Resistor_SMD:R_0402_1005Metric
- R7: value R_US -> 1.2K; footprint Resistor_SMD:R_0603_1608Metric -> Resistor_SMD:R_0402_1005Metric
- R8: value R_US -> 62; footprint Resistor_SMD:R_0603_1608Metric -> Resistor_SMD:R_0402_1005Metric
- R9: value 2K -> 590K; footprint Resistor_SMD:R_0603_1608Metric -> Resistor_SMD:R_0402_1005Metric
- U1: value TL972 -> TPS7A2033PDBVR; footprint Package_SO:SOIC-8_3.9x4.9mm_P1.27mm -> Package_TO_SOT_SMD:SOT-23-5
- U2: value MCP73811T-420I-OT -> TPS63020DSJR; footprint Package_TO_SOT_SMD:SOT-23-5 -> Package_SON:VSON-14-1EP_3x4.45mm_P0.65mm_EP1.6x4.2mm
- moved J4 113.0 mm to (99.0, 70.2)
- moved R5 101.6 mm to (100.0, 63.2), turned to 90 degrees
- moved R6 99.2 mm to (100.0, 60.8)
- moved R2 92.8 mm to (110.0, 66.5), turned to 90 degrees
- moved R4 92.3 mm to (113.5, 60.2), turned to 0 degrees
- moved R3 89.7 mm to (113.5, 61.2), turned to 0 degrees
- moved R8 77.1 mm to (128.8, 57.2), turned to 90 degrees
- moved R1 73.7 mm to (120.0, 68.5), turned to 0 degrees
- moved R7 71.5 mm to (130.2, 57.8)
- moved C1 69.2 mm to (153.3, 53.2), turned to 180 degrees
- moved C2 62.2 mm to (162.1, 53.5)
- moved J3 61.4 mm to (183.7, 51.2), turned to -90 degrees
- moved U2 48.1 mm to (181.6, 62.8)
- moved R9 47.1 mm to (177.8, 62.3), turned to 180 degrees
- moved U1 37.0 mm to (168.2, 68.0), turned to 0 degrees
Connections:
- C1 pad 1: Net-(J3-Pin_1) -> BATT_SENSE
- C2 pad 1: Net-(D1-K) -> GND
- C2 pad 2: GND -> NRST
- J3 pad 1: Net-(J3-Pin_1) -> GND
- J3 pad 2: Net-(A1-VIN) -> /bat+
- J4 pad 1: Net-(J3-Pin_1) -> /out
- J4 pad 2: GND -> Net-(J4-Pin_2)
- R1 pad 1: Net-(J1-Pin_1) -> 3V45_D
- R1 pad 2: /3V3_A -> I2C1_SDA
- R2 pad 1: Net-(J2-Pin_1) -> 3V45_D
- R2 pad 2: /3V3_A -> I2C1_SCL
- R3 pad 2: Net-(U1B--) -> Net-(U3-ADDR0_SCLK)
- R4 pad 2: Net-(U1A--) -> Net-(U3-ADDR1_MISO)
- R5 pad 1: Net-(J2-Pin_1) -> 3V45_D
- R5 pad 2: GND -> Net-(U4-ADDR0_SCLK)
- R6 pad 1: Net-(J1-Pin_1) -> GND
- R6 pad 2: GND -> Net-(U4-ADDR1_MISO)
- R7 pad 1: Net-(U1B--) -> Net-(U6-OUTL)
- R7 pad 2: Net-(A1-AUDIO_IN_R) -> Net-(R7-Pad2)
- R8 pad 1: Net-(U1A--) -> Net-(R7-Pad2)
- R8 pad 2: Net-(A1-AUDIO_IN_L) -> GND
- R9 pad 1: GND -> Net-(U2-FB)
- R9 pad 2: Net-(U2-PROG) -> 3V45_D
- U1 pad 1: Net-(A1-AUDIO_IN_L) -> 3V45_D
- U1 pad 2: Net-(U1A--) -> GND
- U1 pad 3: Net-(J1-Pin_1) -> 3V45_D
- U1 pad 4: GND -> unconnected-(U1-NC-Pad4)
- U1 pad 5: Net-(J2-Pin_1) -> 3V3_A
- U2 pad 1: Net-(D1-K) -> VBAT
- U2 pad 3: Net-(J3-Pin_1) -> Net-(U2-FB)
- U2 pad 4: unconnected-(U2-VDD-Pad4) -> 3V45_D
- U2 pad 5: Net-(U2-PROG) -> 3V45_D
Routing:
- net Net-(A1-AUDIO_IN_R): track 41.2 -> 0.00 mm, vias 2 -> 0
- net Net-(J3-Pin_4): track 34.7 -> 0.00 mm
- net Net-(D1-A): track 33.9 -> 0.00 mm
- net Net-(A1-AUDIO_IN_L): track 28.3 -> 0.00 mm, vias 2 -> 0
- net Net-(J1-Pin_1): track 30.1 -> 1.78 mm
- net Net-(A1-VIN): track 27.3 -> 0.00 mm, vias 1 -> 0
- net Net-(A1-AUDIO_OUT_L): track 26.1 -> 0.00 mm
- net Net-(J3-Pin_1): track 19.7 -> 0.00 mm
- net Net-(J2-Pin_1): track 15.7 -> 1.58 mm
- net GND: track 48.7 -> 36.0 mm, vias 7 -> 39
- net 3V45_D: track 0.00 -> 12.5 mm
- net /3V3_A: track 11.0 -> 0.00 mm, vias 5 -> 0
- net CODEC_SHDNZ: track 0.00 -> 9.93 mm, vias 0 -> 1
- net Net-(U7-PH1): track 0.00 -> 7.12 mm
- net Net-(U4-IN4P_GPI4): track 0.00 -> 6.59 mm
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- removed copper zone on In2.Cu, net /3V3_A
Other:
- board size 25 x 55.8 mm -> 90.5 x 30.8 mm

Commit message: WIP
Parts:
- removed C102: 100nF, Capacitor_SMD:C_0402_1005Metric
- removed C103: 1uF, Capacitor_SMD:C_0402_1005Metric
- added C104: 4.7uF, Capacitor_SMD:C_0402_1005Metric, F.Cu at (160.0, 84.5)
- added FB1: 600, Inductor_SMD:L_0603_1608Metric, F.Cu at (158.5, 97.8)
- added RV3: ~, Potentiometer_THT:Potentiometer_Chinese_Single_Horizontal_Switch, F.Cu at (174.6, 98.8)
- RV1, RV2: footprint Resistor_SMD:R_0402_1005Metric -> Potentiometer_THT:Potentiometer_Alps_RK097_Single_Horizontal
- moved R15 184.1 mm to (0.95, 0.49)
- moved RV2 52.5 mm to (104.8, 98.8), turned to 90 degrees
- moved R2 49.4 mm to (154.2, 88.5), turned to 180 degrees
- moved C37 45.0 mm to (160.5, 95.2)
- moved C38 43.9 mm to (163.0, 95.2)
- moved R1 41.4 mm to (156.2, 88.5), turned to 180 degrees
- moved C10 40.3 mm to (118.2, 95.2)
- moved C11 40.3 mm to (128.5, 93.8)
- moved C12 40.3 mm to (118.2, 97.2)
- moved C13 40.3 mm to (120.8, 91.5)
- moved C14 40.3 mm to (128.5, 92.5)
- moved C7 40.3 mm to (118.2, 93.2)
- moved R7 40.3 mm to (118.2, 96.2)
- moved R8 40.3 mm to (116.8, 95.8)
- moved U6 40.3 mm to (123.2, 95.5)
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Connections:
- Y1 pad 1: Net-(U7-PH0) -> Net-(U7-PH1)
- Y1 pad 2: GND -> Net-(U7-PH0)
- Y1 pad 3: Net-(U7-PH1) -> (no net)
- Y1 pad 4: GND -> (no net)
Routing:
- net 3V45_D: track 12.5 -> 24.5 mm, vias 0 -> 7
- net GND: track 36.0 -> 46.9 mm, vias 39 -> 43
- net I2C1_SCL: track 4.51 -> 8.55 mm
- net Net-(U7-VLXSMPS): track 0.88 -> 4.61 mm
- net I2C1_SDA: track 3.62 -> 7.05 mm
- net Net-(U7-PH0): track 5.54 -> 8.03 mm
- net NRST: track 5.59 -> 3.46 mm
- net BATT_SENSE: track 3.42 -> 2.03 mm
- net Net-(U7-BOOT0): track 1.69 -> 2.51 mm
- net Net-(U7-VFBSMPS): track 6.22 -> 6.88 mm
- added copper zone on In2.Cu, net 3V45_D
Other:
- board size 90.5 x 30.8 mm -> 89 x 29.8 mm

Commit message: WIP
Parts:
- added C105: 4.7uF, Capacitor_SMD:C_0805_2012Metric, F.Cu at (155.7, 91.2)
- added C27: 10uF, Capacitor_SMD:C_0805_2012Metric, F.Cu at (122.0, 91.3)
- added C39: .1uF, Capacitor_SMD:C_0402_1005Metric, F.Cu at (160.0, 85.0)
- added C40: 10uF, Capacitor_SMD:C_0805_2012Metric, F.Cu at (161.2, 89.3)
- added C41: 1uF, Capacitor_SMD:C_0402_1005Metric, F.Cu at (112.8, 83.8)
- added C42: 47uF, Capacitor_SMD:C_0805_2012Metric, F.Cu at (164.9, 87.2)
- added C43: 10uF, Capacitor_SMD:C_0805_2012Metric, F.Cu at (115.5, 86.0)
- added C44: .1uF, Capacitor_SMD:C_0402_1005Metric, F.Cu at (109.1, 89.8)
- added C45: .1uF, Capacitor_SMD:C_0402_1005Metric, F.Cu at (128.5, 89.2)
- added C46: 1uF, Capacitor_SMD:C_0402_1005Metric, F.Cu at (119.5, 83.3)
- added C47: 100nF, Capacitor_SMD:C_0402_1005Metric, F.Cu at (119.5, 82.3)
- added C48: 1uF, Capacitor_SMD:C_0402_1005Metric, F.Cu at (104.5, 90.7)
- added C49: 1uF, Capacitor_SMD:C_0402_1005Metric, F.Cu at (120.5, 89.0)
- added D3: BAS316, Diode_SMD:D_SOD-323, F.Cu at (128.5, 78.5)
- added D4: BAS316, Diode_SMD:D_SOD-323, F.Cu at (124.0, 78.5)
- added D5: BAS316, Diode_SMD:D_SOD-323, F.Cu at (119.5, 78.5)
- added D6: BAS316, Diode_SMD:D_SOD-323, F.Cu at (114.0, 78.5)
- added D7: BAS316, Diode_SMD:D_SOD-323, F.Cu at (109.5, 78.5)
- added D8: BAS316, Diode_SMD:D_SOD-323, F.Cu at (105.0, 78.5)
- added D9: BAS316, Diode_SMD:D_SOD-323, F.Cu at (100.5, 78.5)
- added J1: Bridge Pickup, Connector_PinHeader_2.54mm:PinHeader_1x06_P2.54mm_Vertical, F.Cu at (133.1, 74.5)
- added J2: Neck Pickup, Connector_PinHeader_2.54mm:PinHeader_1x06_P2.54mm_Vertical, F.Cu at (112.5, 74.5)
- added J5: Debug Connector, Connector_PinHeader_1.27mm:PinHeader_2x05_P1.27mm_Vertical, F.Cu at (151.6, 98.4)
- C1: value C -> .1uF
- C101, C104: value 4.7uF -> 100nF
- Y1: value 24.576MHz -> 24.576
- moved R15 162.2 mm to (145.2, 74.5)
- moved J4 69.5 mm to (169.0, 97.8), turned to -90 degrees
- moved U1 46.3 mm to (115.8, 83.2), turned to 180 degrees
- moved FB1 21.7 mm to (149.5, 78.0)
- moved C23 20.6 mm to (167.8, 95.2), turned to 0 degrees
- moved C38 19.8 mm to (150.0, 80.2)
- moved C37 19.1 mm to (150.0, 79.2)
- moved U8 18.7 mm to (165.0, 93.0), turned to 90 degrees
- moved R17 17.1 mm to (162.8, 93.0), turned to 90 degrees
- moved C30 15.2 mm to (167.2, 93.0), turned to -90 degrees
- moved J3 13.8 mm to (167.9, 75.8)
- moved C11 12.4 mm to (117.5, 99.5), turned to 180 degrees
- moved C95 11.4 mm to (154.7, 88.2)
- moved L2 11.2 mm to (152.7, 88.4), turned to 180 degrees
- moved C104 10.9 mm to (151.2, 90.9)
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Connections:
- C4 pad 1: Net-(U3-IN1P_GPI1) -> Net-(D2-K)
- C4 pad 2: Net-(J1-Pin_3) -> Net-(D2-A)
- D2 pad 1: unconnected-(D2-K-Pad1) -> Net-(D2-K)
- D2 pad 2: unconnected-(D2-A-Pad2) -> Net-(D2-A)
- U3 pad 6: Net-(U3-IN1P_GPI1) -> Net-(D2-K)
- Y1 pad 1: Net-(U7-PH1) -> Net-(U7-PH0)
- Y1 pad 2: Net-(U7-PH0) -> GND
- Y1 pad 3: (no net) -> Net-(U7-PH1)
- Y1 pad 4: (no net) -> GND
Routing:
- net 3V45_D: track 24.5 -> 152.5 mm, vias 7 -> 16
- net 3V3_A: track 2.83 -> 124.5 mm
- net Net-(R7-Pad2): track 0.99 -> 84.8 mm, vias 0 -> 4
- net GND: track 46.9 -> 128.9 mm, vias 43 -> 105
- net SAI4_SD_B: track 0.00 -> 73.5 mm, vias 0 -> 6
- net SAI4_SCK_B: track 0.00 -> 68.7 mm, vias 0 -> 6
- net SAI4_FS_B: track 0.00 -> 68.7 mm, vias 0 -> 5
- net I2C1_SCL: track 8.55 -> 74.2 mm, vias 1 -> 3
- net I2C1_SDA: track 7.05 -> 72.2 mm, vias 1 -> 5
- net VBAT: track 5.01 -> 58.1 mm, vias 0 -> 4
- net Pot3: track 0.00 -> 49.2 mm, vias 0 -> 2
- net I2S1_CK: track 0.00 -> 48.1 mm, vias 0 -> 4
- net I2S1_SDO: track 0.00 -> 46.2 mm, vias 0 -> 4
- net I2S1_WS: track 0.00 -> 44.5 mm, vias 0 -> 4
- net /MCU/USART3_TX: track 0.00 -> 37.3 mm, vias 0 -> 1
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Other:
- board text added: "Lines for the BT module"
