File: Onboard DSP Board HW/Main Board/Main Board.kicad_pcb (KiCad board)
At the start: 4 copper layers, 89 x 29.8 mm, 106 parts, among them J1 Bridge Pickup, J2 Neck Pickup, J3 Battery, J4 Output Jack, J5 Debug Connector, U1 TPS7A2033PDBVR, U2 TPS63020DSJR, U3 XLV320ADC5140IRTWR, U4 XLV320ADC5140IRTWR, U6 PCM5102, U7 STM32H725RGVx, U8 TP4054, Y1 24.576

Commit message: WIP
Parts:
- added D1: LED, LED_SMD:LED_0603_1608Metric, F.Cu at (142.7, 74.5)
- Y1: value 24.576 -> 24Mhz; footprint Crystal:Crystal_SMD_3225-4Pin_3.2x2.5mm -> Crystal:Crystal_SMD_WE_IQXC-26-4Pin_1.6x1.2mm
- moved C93 2.06 mm to (154.8, 85.0)
- moved C94 1.47 mm to (153.3, 82.2)
- moved Y1 1.36 mm to (153.1, 84.0)
- moved C2 1.00 mm to (151.8, 81.7)
Routing:
- net (no net): track 0.00 -> 24.6 mm
- net Net-(U7-PH1): track 8.36 -> 5.72 mm
- net NRST: track 28.3 -> 25.7 mm
- net GND: track 128.9 -> 126.8 mm, vias 105 -> 106
- net Net-(U7-PH0): track 8.04 -> 6.39 mm
- net Net-(D1-K): track 0.00 -> 1.23 mm

Commit message: WIP
Parts:
- added U5: E104-BT5032A, E104_BT5032A:WIRELM-SMD_E104-BT5010A, F.Cu at (176.1, 82.2)
- moved J3 2.01 mm to (165.9, 75.6)
- moved C39 1.90 mm to (158.1, 85.0)
- moved C40 1.90 mm to (159.3, 89.3)
- moved L1 1.90 mm to (166.7, 83.8)
- moved R10 1.90 mm to (167.6, 88.2)
- moved R11 1.90 mm to (157.9, 82.1)
- moved R9 1.90 mm to (166.6, 88.2)
- moved U2 1.90 mm to (161.4, 83.8)
- moved C42 1.90 mm to (163.1, 87.2)
Connections:
- U7 pad 36: /MCU/BT1 -> unconnected-(U7-PB12-Pad36)
- U7 pad 37: /MCU/USART3_CTS -> UART3_CTS
- U7 pad 38: /MCU/USART3_RTS -> UART3_RTS
- U7 pad 39: /MCU/BT2 -> unconnected-(U7-PB15-Pad39)
- U7 pad 54: /MCU/USART3_TX -> UART3_TX
- U7 pad 55: /MCU/USART3_RX -> UART3_RX
Routing:
- net UART3_RX: track 0.00 -> 51.2 mm, vias 0 -> 4
- net UART3_CTS: track 0.00 -> 51.2 mm, vias 0 -> 4
- net UART3_TX: track 0.00 -> 50.5 mm, vias 0 -> 2
- net UART3_RTS: track 0.00 -> 45.7 mm, vias 0 -> 2
- net /MCU/USART3_TX: track 37.3 -> 0.00 mm, vias 1 -> 0
- net /MCU/USART3_RX: track 36.3 -> 0.00 mm, vias 1 -> 0
- net /MCU/USART3_CTS: track 24.7 -> 0.00 mm, vias 1 -> 0
- net (no net): track 24.6 -> 0.00 mm
- net /MCU/USART3_RTS: track 22.9 -> 0.00 mm, vias 1 -> 0
- net 3V45_D: track 152.5 -> 173.6 mm
- net GND: track 126.8 -> 131.1 mm, vias 106 -> 109
- net /bat+: track 30.2 -> 31.1 mm
Other:
- board text removed: "Lines for the BT module"

Commit message: WIP
Parts:
- RV3: value ~ -> 10K
- moved C90 0.71 mm to (142.2, 81.4), turned to 180 degrees
Connections:
- U7 pad 32: unconnected-(U7-PB10-Pad32) -> LED
- U7 pad 57: LED -> unconnected-(U7-PD2-Pad57)
Routing:
- net LED: track 0.00 -> 9.03 mm, vias 0 -> 2
- net GND: track 131.1 -> 132.2 mm, vias 109 -> 110
Changed lines of the file:
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@@
 			)
 		)
-		(property "Value" "~"
+		(property "Value" "10K"
 			(at -7.5 -4.4 90)
 			(layer "F.Fab")
@@
 	(footprint "Capacitor_SMD:C_0402_1005Metric"
 		(layer "F.Cu")
-		(at 142.75 80.93 90)
+		(at 142.22 81.4 180)
 		(descr "Capacitor SMD 0402 (1005 Metric), square (rectangular) end terminal, IPC-7351 nominal, (Body size source: IPC-SM-782 page 76, https://www.pcb-3d.com/wordpress/wp-content/uploads/ipc-sm-782a_amendment_1_and_2.pdf)")
 		(tags "capacitor")
 		(property "Reference" "C90"
-			(at 0 -1.16 90)
+			(at 0 -1.16 0)
 			(layer "F.Fab")
 			(effects
@@
 		)
 		(property "Value" "100nF"
-			(at 0 1.16 90)
+			(at 0 1.16 0)
 			(layer "F.Fab")
 			(effects
@@
 		)
 		(property "Datasheet" "~"
-			(at 0 0 90)
+			(at 0 0 0)
 			(layer "F.Fab")
 			(hide yes)
@@
 		)
 		(property "Description" "Ceramic capacitor — one per VCAP pin (LDO disabled on VFQFPN68, AN5419)"
-			(at 0 0 90)
+			(at 0 0 0)
 			(layer "F.Fab")
 			(hide yes)
@@
 		(duplicate_pad_numbers_are_jumpers no)
 		(fp_line
-			(start -0.107836 -0.36)
-			(end 0.107836 -0.36)
+			(start -0.107836 0.36)
+			(end 0.107836 0.36)
 			(stroke
 				(width 0.12)
@@
 		)
 		(fp_line
-			(start -0.107836 0.36)
-			(end 0.107836 0.36)
+			(start -0.107836 -0.36)
+			(end 0.107836 -0.36)
 			(stroke
 				(width 0.12)
@@
 		)
 		(fp_text user "${REFERENCE}"
-			(at 0 0 90)
+			(at 0 0 0)
 			(layer "F.Fab")
 			(effects
@@
 		)
 		(pad "1" smd roundrect
-			(at -0.48 0 90)
+			(at -0.48 0 180)
 			(size 0.56 0.62)
 			(layers "F.Cu" "F.Mask" "F.Paste")
@@
 		)
 		(pad "2" smd roundrect
-			(at 0.48 0 90)
+			(at 0.48 0 180)
 			(size 0.56 0.62)
 			(layers "F.Cu" "F.Mask" "F.Paste")
@@
 			(layers "F.Cu" "F.Mask" "F.Paste")
 			(roundrect_rratio 0.25)
-			(net "unconnected-(U7-PB10-Pad32)")
+			(net "LED")
 			(pinfunction "PB10_32")
 			(pintype "bidirectional")
@@
 			(layers "F.Cu" "F.Mask" "F.Paste")
 			(roundrect_rratio 0.25)
-			(net "LED")
+			(net "unconnected-(U7-PD2-Pad57)")
 			(pinfunction "PD2_57")
 			(pintype "bidirectional")
@@
 	)
 	(segment
+		(start 145.75 74.5)
+		(end 146.65 74.5)
+		(width 0.2)
+		(layer "F.Cu")
+		(net "GND")
+	)
+	(segment
 		(start 147.270272 79.554103)
 		(end 147.074375 79.75)
@@
 	)
 	(segment
-		(start 142.75 80.45)
-		(end 141.9 80.45)
-		(width 0.5)
-		(layer "F.Cu")
-		(net "GND")
-	)
-	(segment
 		(start 167.25 93.48)
 		(end 167.25 94.25)
@@
 	)
 	(segment
+		(start 146.65 74.5)
+		(end 146.7 74.55)
+		(width 0.2)
+		(layer "F.Cu")
+		(net "GND")
+	)
+	(segment
 		(start 138.99 85.5)
 		(end 138.25 85.5)
@@
 	)
 	(segment
+		(start 141.74 81.4)
+		(end 141.74 80.505985)
+		(width 0.2)
+		(layer "F.Cu")
+		(net "GND")
+	)
+	(segment
 		(start 168.23 95.25)
 		(end 168.23 94.73)
@@
 	)
 	(segment
+		(start 141.74 80.505985)
+		(end 141.795985 80.45)
+		(width 0.2)
+		(layer "F.Cu")
+		(net "GND")
+	)
+	(segment
 		(start 142.55 82.8625)
 		(end 142.55 82.85)
@@
 	)
 	(via
+		(at 141.795985 80.45)
+		(size 0.6)
+		(drill 0.3)
+		(layers "F.Cu" "B.Cu")
+		(net "GND")
+	)
+	(via
 		(at 144.55 84.15)
 		(size 0.6)
@@
 	)
 	(via
-		(at 141.9 80.45)
+		(at 130.2 86.025)
 		(size 0.6)
 		(drill 0.3)
@@
 	)
 	(via
-		(at 130.2 86.025)
+		(at 147.270272 79.554103)
 		(size 0.6)
 		(drill 0.3)
@@
 	)
 	(via
-		(at 147.270272 79.554103)
+		(at 145.75 88.95)
 		(size 0.6)
 		(drill 0.3)
@@
 	)
 	(via
-		(at 145.75 88.95)
+		(at 146.7 74.55)
 		(size 0.6)
 		(drill 0.3)
@@
 	)
 	(segment
-		(start 181.85 80.88)
-		(end 180.78 80.88)
-		(width 0.25)
-		(layer "F.Cu")
-		(net "UART3_RTS")
-	)
-	(segment
-		(start 140.9 84.75)
-		(end 140.75 84.9)
-		(width 0.2)
-		(layer "F.Cu")
-		(net "UART3_RTS")
-	)
-	(segment
-		(start 141.8625 84.75)
-		(end 140.9 84.75)
-		(width 0.2)
-		(layer "F.Cu")
-		(net "UART3_RTS")
-	)
-	(segment
-		(start 180.78 80.88)
-		(end 179.9 80)
-		(width 0.25)
-		(layer "F.Cu")
-		(net "UART3_RTS")
-	)
-	(via
-		(at 179.9 80)
-		(size 0.6)
-		(drill 0.3)
-		(layers "F.Cu" "B.Cu")
-		(net "UART3_RTS")
-	)
-	(via
-		(at 140.75 84.9)
-		(size 0.6)
-		(drill 0.3)
-		(layers "F.Cu" "B.Cu")
-		(net "UART3_RTS")
-	)
-	(segment
-		(start 142.9 81.35)
-		(end 143.831855 81.35)
-		(width 0.2)
-		(layer "B.Cu")
-		(net "UART3_RTS")
-	)
-	(segment
-		(start 152.895897 80.104103)
-		(end 153.3 79.7)
-		(width 0.2)
-		(layer "B.Cu")
-		(net "UART3_RTS")
-	)
-	(segment
-		(start 143.831855 81.35)
-		(end 145.077752 80.104103)
-		(width 0.2)
-		(layer "B.Cu")
-		(net "UART3_RTS")
-	)
-	(segment
-		(start 140.75 84.9)
-		(end 140.75 83.5)
-		(width 0.2)
-		(layer "B.Cu")
-		(net "UART3_RTS")
-	)
-	(segment
-		(start 179.6 79.7)
-		(end 179.9 80)
-		(width 0.2)
-		(layer "B.Cu")
-		(net "UART3_RTS")
-	)
-	(segment
-		(start 140.75 83.5)
-		(end 142.9 81.35)
-		(width 0.2)
-		(layer "B.Cu")
-		(net "UART3_RTS")
-	)
-	(segment
-		(start 145.077752 80.104103)
-		(end 152.895897 80.104103)
-		(width 0.2)
-		(layer "B.Cu")
-		(net "UART3_RTS")
-	)
-	(segment
-		(start 153.3 79.7)
-		(end 179.6 79.7)
-		(width 0.2)
-		(layer "B.Cu")
-		(net "UART3_RTS")
-	)
-	(segment
 		(start 174.25 79.25)
 		(end 175.35 80.35)
@@
 	)
 	(segment
+		(start 181.85 80.88)
+		(end 180.78 80.88)
+		(width 0.25)
+		(layer "F.Cu")
+		(net "UART3_RTS")
+	)
+	(segment
+		(start 140.9 84.75)
+		(end 140.75 84.9)
+		(width 0.2)
+		(layer "F.Cu")
+		(net "UART3_RTS")
+	)
+	(segment
+		(start 141.8625 84.75)
+		(end 140.9 84.75)
+		(width 0.2)
+		(layer "F.Cu")
+		(net "UART3_RTS")
+	)
+	(segment
+		(start 180.78 80.88)
+		(end 179.9 80)
+		(width 0.25)
+		(layer "F.Cu")
+		(net "UART3_RTS")
+	)
+	(via
+		(at 179.9 80)
+		(size 0.6)
+		(drill 0.3)
+		(layers "F.Cu" "B.Cu")
+		(net "UART3_RTS")
+	)
+	(via
+		(at 140.75 84.9)
+		(size 0.6)
+		(drill 0.3)
+		(layers "F.Cu" "B.Cu")
+		(net "UART3_RTS")
+	)
+	(segment
+		(start 142.9 81.35)
+		(end 143.831855 81.35)
+		(width 0.2)
+		(layer "B.Cu")
+		(net "UART3_RTS")
+	)
+	(segment
+		(start 152.895897 80.104103)
+		(end 153.3 79.7)
+		(width 0.2)
+		(layer "B.Cu")
+		(net "UART3_RTS")
+	)
+	(segment
+		(start 143.831855 81.35)
+		(end 145.077752 80.104103)
+		(width 0.2)
+		(layer "B.Cu")
+		(net "UART3_RTS")
+	)
+	(segment
+		(start 140.75 84.9)
+		(end 140.75 83.5)
+		(width 0.2)
+		(layer "B.Cu")
+		(net "UART3_RTS")
+	)
+	(segment
+		(start 179.6 79.7)
+		(end 179.9 80)
+		(width 0.2)
+		(layer "B.Cu")
+		(net "UART3_RTS")
+	)
+	(segment
+		(start 140.75 83.5)
+		(end 142.9 81.35)
+		(width 0.2)
+		(layer "B.Cu")
+		(net "UART3_RTS")
+	)
+	(segment
+		(start 145.077752 80.104103)
+		(end 152.895897 80.104103)
+		(width 0.2)
+		(layer "B.Cu")
+		(net "UART3_RTS")
+	)
+	(segment
+		(start 153.3 79.7)
+		(end 179.6 79.7)
+		(width 0.2)
+		(layer "B.Cu")
+		(net "UART3_RTS")
+	)
+	(segment
 		(start 151 83)
 		(end 151 81.75)
@@
 	)
 	(segment
+		(start 142.615424 80.45)
+		(end 142.545988 80.45)
+		(width 0.2)
+		(layer "F.Cu")
+		(net "LED")
+	)
+	(segment
+		(start 141.883976 74.541024)
+		(end 141.925 74.5)
+		(width 0.2)
+		(layer "F.Cu")
+		(net "LED")
+	)
+	(segment
+		(start 143.35 81.184576)
+		(end 142.615424 80.45)
+		(width 0.2)
+		(layer "F.Cu")
+		(net "LED")
+	)
+	(segment
+		(start 141.883976 75.663705)
+		(end 141.883976 74.541024)
+		(width 0.2)
+		(layer "F.Cu")
+		(net "LED")
+	)
+	(segment
+		(start 143.35 82.8625)
+		(end 143.35 81.184576)
+		(width 0.2)
+		(layer "F.Cu")
+		(net "LED")
+	)
+	(via
+		(at 142.545988 80.45)
+		(size 0.6)
+		(drill 0.3)
+		(layers "F.Cu" "B.Cu")
+		(net "LED")
+	)
+	(via
+		(at 141.883976 75.663705)
+		(size 0.6)
+		(drill 0.3)
+		(layers "F.Cu" "B.Cu")
+		(net "LED")
+	)
+	(segment
+		(start 142.545988 80.45)
+		(end 142.545988 76.325717)
+		(width 0.2)
+		(layer "B.Cu")
+		(net "LED")
+	)
+	(segment
+		(start 142.545988 76.325717)
+		(end 141.883976 75.663705)
+		(width 0.2)
+		(layer "B.Cu")
+		(net "LED")
+	)
+	(segment

Commit message: WIP
Parts:
- moved C90 0.84 mm to (141.4, 81.7)
- moved C100 0.35 mm to (147.6, 80.8)
Connections:
- U7 pad 14: Pot2 -> unconnected-(U7-PC1-Pad14)
- U7 pad 29: unconnected-(U7-PB0-Pad29) -> Pot2
Routing:
- net Pot3: track 49.2 -> 51.4 mm, vias 2 -> 0
- net Pot2: track 29.7 -> 31.9 mm
- net BATT_SENSE: track 6.08 -> 5.48 mm

Commit message: WIP on FET preamp
Routing:
- net Net-(U7-PA8): track 0.00 -> 2.48 mm, vias 0 -> 1

Commit message: Add JFET preamp to project
Routing:
- added copper zone on B.Cu, net (none)
- added copper zone on F.Cu, net (none)
Changed lines of the file:
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@@
+	)
+	(zone
+		(layers "F.Cu" "B.Cu")
+		(hatch edge 0.5)
+		(priority 2)
+		(connect_pads
+			(clearance 0.2)
+		)
+		(min_thickness 0.25)
+		(fill yes
+			(thermal_gap 0.5)
+			(thermal_bridge_width 0.5)
+			(island_removal_mode 1)
+		)
+		(polygon
+			(pts
+				(xy 92.95 70.55) (xy 92.55 70.8) (xy 91.95 105) (xy 186.7 104.3) (xy 185.55 69.25) (xy 93.3 69.65)
+			)
+		)
 	)
 	(zone

Commit message: WIP on DSP, add connectors
Parts:
- removed C15, C16, C17, C22, C24, C25, C26, C9: 4.7uF, Capacitor_SMD:C_0402_1005Metric
- removed C18, C19, C20, C21, C4, C5, C6, C8: 4.7uF, Capacitor_SMD:C_1206_3216Metric
- removed C35, C36: 1uF, Capacitor_SMD:C_0402_1005Metric
- removed D2, D3, D4, D5, D6, D7, D8, D9: BAS316, Diode_SMD:D_SOD-323
- added C3: 10uF, Capacitor_SMD:C_1206_3216Metric, F.Cu at (115.0, 78.2)
- added R16: 10K, Resistor_SMD:R_0402_1005Metric, F.Cu at (114.0, 80.1)
- added R19: 43K, Resistor_SMD:R_0402_1005Metric, F.Cu at (116.3, 80.1)
- added U9: TLV9001IDCK, Package_TO_SOT_SMD:SOT-353_SC-70-5, F.Cu at (114.9, 75.6)
- J1: footprint Connector_PinHeader_2.54mm:PinHeader_1x06_P2.54mm_Vertical -> Connector_PinHeader_2.00mm:PinHeader_1x07_P2.00mm_Horizontal
- J2: value Neck Pickup -> Bridge Pickup; footprint Connector_PinHeader_2.54mm:PinHeader_1x06_P2.54mm_Vertical -> Connector_PinHeader_2.00mm:PinHeader_1x07_P2.00mm_Horizontal
- moved J2 17.3 mm to (96.7, 81.3), turned to 90 degrees
- moved J1 13.3 mm to (121.8, 81.4), turned to 90 degrees
- moved C41 1.31 mm to (111.5, 83.3)
- moved U1 1.31 mm to (114.5, 82.8)
- moved C46 1.31 mm to (118.2, 82.9)
- moved C47 1.31 mm to (118.2, 81.9)
- moved C33 0.15 mm to (109.9, 88.8)
Connections:
- J1 pad 1: Net-(J1-Pin_1) -> GND
- J1 pad 2: GND -> Net-(J1-Pin_2)
- J1 pad 3: Net-(D2-A) -> Net-(J1-Pin_3)
- J1 pad 4: Net-(D3-A) -> Net-(J1-Pin_4)
- J1 pad 5: Net-(D4-A) -> Net-(J1-Pin_5)
- J1 pad 6: Net-(D5-A) -> /Bias
- J2 pad 1: Net-(J2-Pin_1) -> GND
- J2 pad 2: GND -> Net-(J2-Pin_2)
- J2 pad 3: Net-(D6-A) -> Net-(J2-Pin_3)
- J2 pad 4: Net-(D7-A) -> Net-(J2-Pin_4)
- J2 pad 5: Net-(D8-A) -> Net-(J2-Pin_5)
- J2 pad 6: Net-(D9-A) -> /Bias
- U3 pad 10: Net-(D4-K) -> Net-(J1-Pin_3)
- U3 pad 11: Net-(U3-IN3M_GPO3) -> /Bias
- U3 pad 12: Net-(D5-K) -> Net-(J1-Pin_2)
- U3 pad 13: Net-(U3-IN4M_GPO4) -> /Bias
- U3 pad 5: Net-(J1-Pin_1) -> unconnected-(U3-MICBIAS-Pad5)
- U3 pad 6: Net-(D2-K) -> Net-(J1-Pin_5)
- U3 pad 7: Net-(U3-IN1M_GPO1) -> /Bias
- U3 pad 8: Net-(D3-K) -> Net-(J1-Pin_4)
- U3 pad 9: Net-(U3-IN2M_GPO2) -> /Bias
- U4 pad 10: Net-(D8-K) -> Net-(J2-Pin_3)
- U4 pad 11: Net-(U4-IN3M_GPO3) -> /Bias
- U4 pad 12: Net-(D9-K) -> Net-(J2-Pin_2)
- U4 pad 13: Net-(U4-IN4M_GPO4) -> /Bias
- U4 pad 5: Net-(J2-Pin_1) -> unconnected-(U4-MICBIAS-Pad5)
- U4 pad 6: Net-(D6-K) -> Net-(J2-Pin_5)
- U4 pad 7: Net-(U4-IN1M_GPO1) -> /Bias
- U4 pad 8: Net-(D7-K) -> Net-(J2-Pin_4)
- U4 pad 9: Net-(U4-IN2M_GPO2) -> /Bias
Routing:
- net /Bias: track 0.00 -> 63.9 mm, vias 0 -> 10
- net Net-(J2-Pin_1): track 18.9 -> 0.00 mm
- net Net-(J1-Pin_1): track 17.8 -> 0.00 mm
- net 3V3_A: track 124.5 -> 137.9 mm
- net Net-(D5-K): track 12.2 -> 0.00 mm
- net Net-(D9-K): track 12.0 -> 0.00 mm
- net Net-(D2-K): track 9.75 -> 0.00 mm
- net Net-(D6-K): track 9.72 -> 0.00 mm
- net Net-(D8-K): track 9.14 -> 0.00 mm
- net Net-(D4-K): track 9.04 -> 0.00 mm
- net Net-(D6-A): track 7.70 -> 0.00 mm
- net Net-(D3-K): track 7.69 -> 0.00 mm
- net Net-(D7-K): track 7.66 -> 0.00 mm
- net Net-(J2-Pin_2): track 0.00 -> 7.64 mm
- net GND: track 132.4 -> 125.3 mm, vias 110 -> 105
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- added copper zone on B.Cu, net GND
- added copper zone on F.Cu, net GND
- added copper zone on In2.Cu, net GND
- removed copper zone on B.Cu, net (none)
- removed copper zone on F.Cu, net (none)
