File: Onboard DSP Board HW/Main Board/Main Board.kicad_pcb (KiCad board)
At the start: 4 copper layers, 89 x 29.8 mm, 90 parts, among them J1 Bridge Pickup, J2 Bridge Pickup, J3 Battery, J4 Output Jack, J5 Debug Connector, U1 TPS7A2033PDBVR, U2 TPS63020DSJR, U3 XLV320ADC5140IRTWR, U4 XLV320ADC5140IRTWR, U5 E104-BT5032A, U6 PCM5102, U7 STM32H725RGVx, U8 TP4054, U9 TLV9001IDCK, Y1 24Mhz

Commit message: WIP
Connections:
- J1 pad 2: Net-(J1-Pin_2) -> /Bias
- J1 pad 3: Net-(J1-Pin_3) -> 3V3_A
- J1 pad 6: /Bias -> Net-(J1-Pin_6)
- J1 pad 7: 3V3_A -> Net-(J1-Pin_7)
- J2 pad 2: Net-(J2-Pin_2) -> /Bias
- J2 pad 3: Net-(J2-Pin_3) -> 3V3_A
- J2 pad 6: /Bias -> Net-(J2-Pin_6)
- J2 pad 7: 3V3_A -> Net-(J2-Pin_7)
- U3 pad 10: Net-(J1-Pin_3) -> Net-(J1-Pin_5)
- U3 pad 12: Net-(J1-Pin_2) -> Net-(J1-Pin_4)
- U3 pad 6: Net-(J1-Pin_5) -> Net-(J1-Pin_7)
- U3 pad 8: Net-(J1-Pin_4) -> Net-(J1-Pin_6)
- U4 pad 10: Net-(J2-Pin_3) -> Net-(J2-Pin_5)
- U4 pad 12: Net-(J2-Pin_2) -> Net-(J2-Pin_4)
- U4 pad 6: Net-(J2-Pin_5) -> Net-(J2-Pin_7)
- U4 pad 8: Net-(J2-Pin_4) -> Net-(J2-Pin_6)
Routing:
- net 3V3_A: track 137.9 -> 160.7 mm
- net Net-(J1-Pin_7): track 0.00 -> 8.87 mm
- net Net-(J1-Pin_6): track 0.00 -> 8.60 mm
- net Net-(J2-Pin_2): track 7.64 -> 0.00 mm
- net Net-(J2-Pin_3): track 6.73 -> 0.00 mm
- net Net-(J2-Pin_7): track 0.00 -> 4.80 mm
- net Net-(J1-Pin_3): track 4.29 -> 0.00 mm
- net Net-(J1-Pin_2): track 4.16 -> 0.00 mm
- net Net-(J2-Pin_6): track 0.00 -> 3.77 mm
- net Net-(J1-Pin_4): track 4.81 -> 7.82 mm
- net Net-(J2-Pin_5): track 7.02 -> 4.06 mm
- net Net-(J1-Pin_5): track 5.64 -> 8.08 mm
- net /Bias: track 63.9 -> 62.2 mm
- net Net-(J2-Pin_4): track 6.16 -> 4.96 mm

Commit message: WIP
Parts:
- added C102: 10uF, Capacitor_SMD:C_0603_1608Metric, F.Cu at (156.7, 88.2)
- added C4: 2.2uF, Capacitor_SMD:C_0402_1005Metric, F.Cu at (159.8, 100.5)
- added C50: 22uF, Capacitor_SMD:C_0805_2012Metric, F.Cu at (163.1, 89.3)
- added R20: 10K, Resistor_SMD:R_0402_1005Metric, F.Cu at (123.2, 99.3)
- added R21: 10K, Resistor_SMD:R_0402_1005Metric, F.Cu at (135.0, 95.6)
- C3: footprint Capacitor_SMD:C_1206_3216Metric -> Capacitor_SMD:C_0805_2012Metric
- C42: value 47uF -> 22uF
- C93, C94: value 15pF -> 6.8pF
- C95: value 4.7uF -> 10uF; footprint Capacitor_SMD:C_0402_1005Metric -> Capacitor_SMD:C_0603_1608Metric
- R1, R2: value R -> 4.7K
- R10: value 100K -> 200K
- R15: value R -> 1K
- R16: value 10K -> 100K
- R17: value 30k -> 3.3K
- R19: value 43K -> 68K
- R3, R4, R5, R6: value R -> 10K
- R8: value 62 -> 470
- R9: value 590K -> 1.1M
- TP12, TP13, TP14: footprint AWV:TestPoint_Plated_Hole_ID4_OD7.0mm -> AWV:TestPoint_Plated_Hole_ID7_OD1.2mm
- U2: footprint Package_SON:VSON-14-1EP_3x4.45mm_P0.65mm_EP1.6x4.2mm -> AWV:DSJ14_2P85X1P58
- U3, U4: value XLV320ADC5140IRTWR -> TLV320ADC5140IRTWR; footprint Package_DFN_QFN:HVQFN-24-1EP_4x4mm_P0.5mm_EP2.1x2.1mm -> AWV:RTW24_4P15X4P15_TEX
- moved TP13 13.2 mm to (133.1, 87.1)
- moved C14 1.35 mm to (121.1, 99.3), turned to 180 degrees
- moved D1 0.70 mm to (142.7, 75.2)
- moved R15 0.70 mm to (145.2, 75.2)
- moved L1 0.64 mm to (166.2, 83.4)
- moved TP14 0.49 mm to (171.2, 92.0)
- moved C95 0.40 mm to (155.1, 88.2)
- moved C3 0.35 mm to (114.9, 77.9), turned to 0 degrees
- moved U2 0.30 mm to (161.4, 83.5)
Connections:
- C100 pad 1: 3V45_D -> 3V3_D
- C101 pad 1: 3V45_D -> 3V3_D
- C104 pad 1: 3V45_D -> 3V3_D
- C105 pad 1: 3V45_D -> 3V3_D
- C14 pad 2: 3V45_D -> 3V3_A
- C3 pad 1: Net-(U9-+) -> GND
- C3 pad 2: GND -> Net-(U9-+)
- C42 pad 2: 3V45_D -> 3V3_D
- C46 pad 2: 3V45_D -> VBAT
- C47 pad 2: 3V45_D -> VBAT
- C48 pad 1: 3V45_D -> 3V3_D
- C49 pad 1: 3V45_D -> 3V3_D
- C96 pad 1: 3V45_D -> 3V3_D
- C97 pad 1: 3V45_D -> 3V3_D
- C98 pad 1: 3V45_D -> 3V3_D
- C99 pad 1: 3V45_D -> 3V3_D
- J5 pad 1: 3V45_D -> 3V3_D
- R1 pad 1: 3V45_D -> 3V3_D
- R2 pad 1: 3V45_D -> 3V3_D
- R4 pad 1: GND -> 3V3_D
- R5 pad 1: 3V45_D -> 3V3_D
- R9 pad 2: 3V45_D -> 3V3_D
- U1 pad 1: 3V45_D -> VBAT
- U1 pad 3: 3V45_D -> VBAT
- U2 pad 4: 3V45_D -> 3V3_D
- U2 pad 5: 3V45_D -> 3V3_D
- U3 pad 19: 3V45_D -> 3V3_D
- U4 pad 19: 3V45_D -> 3V3_D
- U5 pad 17: 3V45_D -> 3V3_D
- U6 pad 20: 3V45_D -> 3V3_A
- U6 pad 7: /To Test Point -> unconnected-(U6-OUTR-Pad7)
- U7 pad 1: 3V45_D -> 3V3_D
- U7 pad 22: 3V45_D -> 3V3_D
- U7 pad 35: 3V45_D -> 3V3_D
- U7 pad 51: 3V45_D -> 3V3_D
- U7 pad 6: 3V45_D -> 3V3_D
- U7 pad 68: 3V45_D -> 3V3_D
- U7 pad 9: 3V45_D -> 3V3_D
Routing:
- net 3V45_D: track 174.4 -> 0.00 mm, vias 16 -> 0
- net 3V3_D: track 0.00 -> 145.6 mm, vias 0 -> 14
- net VBAT: track 58.1 -> 122.2 mm, vias 4 -> 7
- net GND: track 125.3 -> 99.1 mm, vias 105 -> 106
- net 3V3_A: track 160.7 -> 170.1 mm
- net Net-(U7-VFBSMPS): track 6.63 -> 8.74 mm
- net NRST: track 25.3 -> 23.2 mm, vias 1 -> 3
- net SAI4_SD_B: track 73.2 -> 74.7 mm
- net DAC_XSMT: track 34.2 -> 35.3 mm, vias 2 -> 3
- net unconnected-(U7-PB5-Pad60): track 0.00 -> 1.03 mm, vias 0 -> 1
- net Pot3: track 51.4 -> 52.3 mm
- net UART3_RX: track 51.2 -> 52.0 mm
- net Net-(L1-Pad2): track 4.04 -> 4.75 mm
- net Net-(U9-+): track 5.78 -> 5.24 mm
- added copper zone on In2.Cu, net 3V3_D
- removed copper zone on In2.Cu, net 3V45_D
