File: Onboard DSP Board HW/Main Board/Main Board.kicad_sch (KiCad schematic)
At the start: 76 parts, among them J1 Bridge Pickup, J2 Neck Pickup, J3 Battery, J4 Output Jack, J5 Debug Connector, U1 TPS7A2033PDBVR, U2 TPS63020DSJR, U3 XLV320ADC5140IRTWR, U4 XLV320ADC5140IRTWR, U6 PCM5102, U8 TP4054

Commit message: WIP
Parts:
- removed TP2, TP3, TP4, TP5, TP6, TP7, TP8, TP9: (no value), symbol Connector:TestPoint
- added D2: BAS316, Diode_SMD:D_SOD-323, symbol Diode:1N914
- added TP12, TP13, TP14: (no value), symbol Connector:TestPoint
- C1, C10, C11, C12, C13, C14, C15, C16, C17, C22, C24, C25, C26, C28, C29, C31, C32, C33, C34, C35, C36, C37, C38, C7, C9: footprint (none) -> Capacitor_SMD:C_0402_1005Metric
- C18, C19, C20, C21, C4, C5, C6, C8: footprint (none) -> Capacitor_SMD:C_1206_3216Metric
- C23, C30: footprint Capacitor_SMD:C_0603_1608Metric -> Capacitor_SMD:C_0402_1005Metric
- L1: footprint (none) -> Inductor_SMD:L_Sunlord_SWPA4030S
- R1, R10, R11, R12, R13, R15, R2, R3, R4, R5, R6, R7, R8, R9, RV1, RV2: footprint (none) -> Resistor_SMD:R_0402_1005Metric
- R17: footprint Resistor_SMD:R_0603_1608Metric -> Resistor_SMD:R_0402_1005Metric
- U2: footprint DSJ14_2P85X1P58 -> Package_SON:VSON-14-1EP_3x4.45mm_P0.65mm_EP1.6x4.2mm
- U3, U4: footprint RTW24_4P15X4P15_TEX -> Package_DFN_QFN:HVQFN-24-1EP_4x4mm_P0.5mm_EP2.1x2.1mm
Connections:
- net GND: now also TP12.1, TP13.1, TP14.1
Other:
- moved on the sheet: C23

Commit message: WIP
Parts:
- RV1, RV2: footprint Resistor_SMD:R_0402_1005Metric -> Potentiometer_THT:Potentiometer_Alps_RK097_Single_Horizontal
Changed lines of the file:
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@@
 			)
 		)
-		(property "Footprint" "Resistor_SMD:R_0402_1005Metric"
+		(property "Footprint" "Potentiometer_THT:Potentiometer_Alps_RK097_Single_Horizontal"
 			(at 294.64 107.95 0)
 			(hide yes)
@@
 			)
 		)
-		(property "Footprint" "Resistor_SMD:R_0402_1005Metric"
+		(property "Footprint" "Potentiometer_THT:Potentiometer_Alps_RK097_Single_Horizontal"
 			(at 316.23 107.95 0)
 			(hide yes)

Commit message: WIP
Parts:
- added C27: 10uF, Capacitor_SMD:C_0805_2012Metric, symbol Device:C
- added C39, C44, C45: .1uF, Capacitor_SMD:C_0402_1005Metric, symbol Device:C_Small
- added C40, C43: 10uF, Capacitor_SMD:C_0805_2012Metric, symbol Device:C_Small
- added C41, C46, C48, C49: 1uF, Capacitor_SMD:C_0402_1005Metric, symbol Device:C_Small
- added C42: 47uF, Capacitor_SMD:C_0805_2012Metric, symbol Device:C_Small
- added C47: 100nF, Capacitor_SMD:C_0402_1005Metric, symbol Device:C_Small
- added D3, D4, D5, D6, D7, D8, D9: BAS316, Diode_SMD:D_SOD-323, symbol Diode:1N914
- C1: value C -> .1uF
- FB1: footprint (none) -> Inductor_SMD:L_0603_1608Metric
- J1, J2: footprint (none) -> Connector_PinHeader_2.54mm:PinHeader_1x06_P2.54mm_Vertical
- J5: footprint (none) -> Connector_PinHeader_1.27mm:PinHeader_2x05_P1.27mm_Vertical
Connections:
- net 3V3_A: now also C27.1, C41.2, C43.1, C44.2, C45.2
- net 3V45_D: now also C42.2, C46.2, C47.2, C48.1, C49.1
- net GND: now also C27.2, C39.1, C40.1, C41.1, C42.1, C43.2, C44.1, C45.1, C46.1, C47.1, C48.2, C49.2
- net VBAT: now also C39.2, C40.2
- net at C20.1, U4.10 (IN3P_GPI3): now also D8.1 (K)
- net at C20.2, J2.5 (Pin_5): now also D8.2 (A)
- net at C5.1, U3.8 (IN2P_GPI2): now also D3.1 (K)
- net at C5.2, J1.4 (Pin_4): now also D3.2 (A)
- net at C4.1, U3.6 (IN1P_GPI1): now also D2.1 (K)
- net at C4.2, J1.3 (Pin_3): now also D2.2 (A)
- net at C18.1, U4.6 (IN1P_GPI1): now also D6.1 (K)
- net at C18.2, J2.3 (Pin_3): now also D6.2 (A)
- net at C6.1, U3.10 (IN3P_GPI3): now also D4.1 (K)
- net at C6.2, J1.5 (Pin_5): now also D4.2 (A)
- net at C8.1, U3.12 (IN4P_GPI4): now also D5.1 (K)
- net at C8.2, J1.6 (Pin_6): now also D5.2 (A)
- net at C21.1, U4.12 (IN4P_GPI4): now also D9.1 (K)
- net at C19.1, U4.8 (IN2P_GPI2): now also D7.1 (K)
- net at C19.2, J2.4 (Pin_4): now also D7.2 (A)
- net at C21.2, J2.6 (Pin_6): now also D9.2 (A)
Other:
- moved on the sheet: C14, C15, C16, C17, C19, C20, C21, C22, C24, C26, C37, C38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

Commit message: WIP
Parts:
- D1: footprint (none) -> LED_SMD:LED_0603_1608Metric
Changed lines of the file:
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@@
 			)
 		)
-		(property "Footprint" ""
+		(property "Footprint" "LED_SMD:LED_0603_1608Metric"
 			(at 248.92 86.36 0)
 			(hide yes)

Commit message: WIP
Parts:
- added U5: E104-BT5032A, E104_BT5032A:WIRELM-SMD_E104-BT5010A, symbol Ebyte:E104-BT5032A
- RV3: value (none) -> 10K
Connections:
- net 3V45_D: now also U5.17 (VCC)
- net GND: now also U5.1 (GND), U5.16 (GND), U5.9 (GND)
- new net UART3_CTS: U5.20 (RTS)
- new net UART3_RTS: U5.21 (CTS)
- new net UART3_RX: U5.19 (TXD)
- new net UART3_TX: U5.18 (RXD)

Commit message: WIP on DSP, add connectors
Parts:
- removed C15, C16, C17, C22, C24, C25, C26, C9: 4.7uF, Capacitor_SMD:C_0402_1005Metric, symbol Device:C_Small
- removed C18, C19, C20, C21, C4, C5, C6, C8: 4.7uF, Capacitor_SMD:C_1206_3216Metric, symbol Device:C_Polarized_Small
- removed C35, C36: 1uF, Capacitor_SMD:C_0402_1005Metric, symbol Device:C_Small
- removed D2, D3, D4, D5, D6, D7, D8, D9: BAS316, Diode_SMD:D_SOD-323, symbol Diode:1N914
- removed J1: Bridge Pickup, Connector_PinHeader_2.54mm:PinHeader_1x06_P2.54mm_Vertical, symbol Connector:Conn_01x06_Socket
- removed J2: Neck Pickup, Connector_PinHeader_2.54mm:PinHeader_1x06_P2.54mm_Vertical, symbol Connector:Conn_01x06_Socket
- removed TP11: (no value), symbol Connector:TestPoint
- added C3: 10uF, Capacitor_SMD:C_1206_3216Metric, symbol Device:C_Polarized_Small
- added J1, J2: Bridge Pickup, Connector_PinHeader_2.00mm:PinHeader_1x07_P2.00mm_Horizontal, symbol Connector:Conn_01x07_Socket
- added R16: 10K, Resistor_SMD:R_0402_1005Metric, symbol Device:R
- added R19: 43K, Resistor_SMD:R_0402_1005Metric, symbol Device:R
- added U9: TLV9001IDCK, Package_TO_SOT_SMD:SOT-353_SC-70-5, symbol Amplifier_Operational:TLV9001IDCK
Connections:
- net 3V3_A: now also J1.7 (Pin_7), J2.7 (Pin_7), R16.1, U9.5 (V+)
- net GND: now also C3.2, J1.1 (Pin_1), J2.1 (Pin_1), R19.2, U9.2 (V-)
- net at U4.10 (IN3P_GPI3): now also J2.3 (Pin_3)
- net at U3.8 (IN2P_GPI2): now also J1.4 (Pin_4)
- net at U3.6 (IN1P_GPI1): now also J1.5 (Pin_5)
- net at U4.6 (IN1P_GPI1): now also J2.5 (Pin_5)
- net Bias: now reaches U3.7 (IN1M_GPO1)
- net Bias: now also U3.11 (IN3M_GPO3), U3.13 (IN4M_GPO4), U3.9 (IN2M_GPO2), U4.11 (IN3M_GPO3), U4.13 (IN4M_GPO4), U4.7 (IN1M_GPO1), U4.9 (IN2M_GPO2), J1.6 (Pin_6), J2.6 (Pin_6), U9.3 (-), U9.4
- net at U3.10 (IN3P_GPI3): now also J1.3 (Pin_3)
- net at U4.12 (IN4P_GPI4): now also J2.2 (Pin_2)
- net at U3.12 (IN4P_GPI4): now also J1.2 (Pin_2)
- net at U4.8 (IN2P_GPI2): now also J2.4 (Pin_4)
- new net: C3.1, R16.2, R19.1, U9.1 (+)
Other:
- moved on the sheet: C31, C43, J5

Commit message: WIP
Parts:
- TP12, TP13, TP14: footprint (none) -> AWV:TestPoint_Plated_Hole_ID4_OD7.0mm
Changed lines of the file:
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@@
 			)
 		)
-		(property "Footprint" ""
+		(property "Footprint" "AWV:TestPoint_Plated_Hole_ID4_OD7.0mm"
 			(at 257.81 133.35 0)
 			(hide yes)
@@
 			)
 		)
-		(property "Footprint" ""
+		(property "Footprint" "AWV:TestPoint_Plated_Hole_ID4_OD7.0mm"
 			(at 270.51 133.35 0)
 			(hide yes)
@@
 			)
 		)
-		(property "Footprint" ""
+		(property "Footprint" "AWV:TestPoint_Plated_Hole_ID4_OD7.0mm"
 			(at 264.16 133.35 0)
 			(hide yes)

Commit message: WIP
Connections:
- net 3V3_A: now also J1.3 (Pin_3), J2.3 (Pin_3); no longer J1.7 (Pin_7), J2.7 (Pin_7)
- net Bias: now also J1.2 (Pin_2), J2.2 (Pin_2); no longer J1.6 (Pin_6), J2.6 (Pin_6)
- net at U3.12 (IN4P_GPI4): now also J1.4 (Pin_4); no longer J1.2 (Pin_2)
- net at U3.10 (IN3P_GPI3): now also J1.5 (Pin_5); no longer J1.3 (Pin_3)
- net at U3.8 (IN2P_GPI2): now also J1.6 (Pin_6); no longer J1.4 (Pin_4)
- net at U3.6 (IN1P_GPI1): now also J1.7 (Pin_7); no longer J1.5 (Pin_5)
- net at U4.12 (IN4P_GPI4): now also J2.4 (Pin_4); no longer J2.2 (Pin_2)
- net at U4.10 (IN3P_GPI3): now also J2.5 (Pin_5); no longer J2.3 (Pin_3)
- net at U4.8 (IN2P_GPI2): now also J2.6 (Pin_6); no longer J2.4 (Pin_4)
- net at U4.6 (IN1P_GPI1): now also J2.7 (Pin_7); no longer J2.5 (Pin_5)
Other:
- moved on the sheet: J2
