File: Onboard DSP Board HW/Main Board/Main Board.kicad_sch (KiCad schematic)
At the start: 69 parts, among them J1 Bridge Pickup, J2 Bridge Pickup, J3 Battery, J4 Output Jack, J5 Debug Connector, U1 TPS7A2033PDBVR, U2 TPS63020DSJR, U3 XLV320ADC5140IRTWR, U4 XLV320ADC5140IRTWR, U5 E104-BT5032A, U6 PCM5102, U8 TP4054, U9 TLV9001IDCK

Commit message: WIP
Parts:
- removed C3: 10uF, Capacitor_SMD:C_1206_3216Metric, symbol Device:C_Polarized_Small
- removed U2: TPS63020DSJR, Package_SON:VSON-14-1EP_3x4.45mm_P0.65mm_EP1.6x4.2mm, symbol TPS63020:TPS63020DSJR
- removed U3, U4: XLV320ADC5140IRTWR, Package_DFN_QFN:HVQFN-24-1EP_4x4mm_P0.5mm_EP2.1x2.1mm, symbol XLV320ADC5140:XLV320ADC5140IRTWR
- added C3: 10uF, Capacitor_SMD:C_0805_2012Metric, symbol Device:C_Small
- added C4: 2.2uF, Capacitor_SMD:C_0402_1005Metric, symbol Device:C_Small
- added C50: 22uF, Capacitor_SMD:C_0805_2012Metric, symbol Device:C_Small
- added R20, R21: 10K, Resistor_SMD:R_0402_1005Metric, symbol Device:R
- added U2: TPS63020DSJR, AWV:DSJ14_2P85X1P58, symbol AWV:TPS63020DSJR
- added U3, U4: TLV320ADC5140IRTWR, AWV:RTW24_4P15X4P15_TEX, symbol AWV:TLV320ADC5140IRTWR
- C42: value 47uF -> 22uF
- D1: LCSC (none) -> C2286
- FB1: LCSC (none) -> C1002
- R1, R2: value R -> 4.7K
- R10: value 100K -> 200K
- R15: value R -> 1K
- R16: value 10K -> 100K
- R17: value 30k -> 3.3K
- R19: value 43K -> 68K
- R3, R4, R5, R6: value R -> 10K
- R8: value 62 -> 470
- R9: value 590K -> 1.1M
- TP12, TP13, TP14: footprint AWV:TestPoint_Plated_Hole_ID4_OD7.0mm -> AWV:TestPoint_Plated_Hole_ID7_OD1.2mm
Connections:
- net 3V3_A: now also C14.2, U6.20 (DVDD), U3.1 (AVDD), U4.1 (AVDD)
- net Bias: now also U3.11 (IN3M_GPO3), U3.13 (IN4M_GPO4), U3.7 (IN1M_GPO1), U3.9 (IN2M_GPO2), U4.11 (IN3M_GPO3), U4.13 (IN4M_GPO4), U4.7 (IN1M_GPO1), U4.9 (IN2M_GPO2)
- net CODEC_SHDNZ: now also U3.14 (SHDNZ), U4.14 (SHDNZ)
- net DAC_XSMT: now also R20.1
- net GND: now also C3.1, C4.2, C50.1, R20.2, R21.2, U2.13 (PS/SYNC), U2.14 (PG), U2.15 (EPAD), U2.2 (GND), U3.25 (EPAD), U3.4 (AVSS), U4.25 (EPAD), U4.4 (AVSS); no longer R4.1
- net I2C1_SCL: now also U3.17 (SCL_MOSI), U4.17 (SCL_MOSI)
- net I2C1_SDA: now also U3.18 (SDA_SSZ), U4.18 (SDA_SSZ)
- net SAI4_FS_B: now also U3.23 (FSYNC), U4.23 (FSYNC)
- net SAI4_SCK_B: now also U3.22 (BCLK), U4.22 (BCLK)
- net SAI4_SD_B: now also R21.1, U3.21 (SDOUT), U4.21 (SDOUT)
- net VBAT: now also C46.2, C47.2, U1.1 (IN), U1.3 (EN), U2.1 (VINA), U2.10 (VIN), U2.11 (VIN), U2.12 (EN)
- net at R7.2, R8.1, RV3.3: now also C4.1
- net at R4.2: now also U3.15 (ADDR1_MISO)
- net at R3.2: now also U3.16 (ADDR0_SCLK)
- net at J1.4 (Pin_4): now also U3.12 (IN4P_GPI4)
- net at J1.5 (Pin_5): now also U3.10 (IN3P_GPI3)
- net at J1.6 (Pin_6): now also U3.8 (IN2P_GPI2)
- net at J1.7 (Pin_7): now also U3.6 (IN1P_GPI1)
- net at R6.2: now also U4.15 (ADDR1_MISO)
- net at R16.2, R19.1, U9.1 (+): now also C3.2
- net at J2.4 (Pin_4): now also U4.12 (IN4P_GPI4)
- net at J2.5 (Pin_5): now also U4.10 (IN3P_GPI3)
- net at J2.6 (Pin_6): now also U4.8 (IN2P_GPI2)
- net at J2.7 (Pin_7): now also U4.6 (IN1P_GPI1)
- net at R5.2: now also U4.16 (ADDR0_SCLK)
- net at C33.2: now also U4.2 (AREG)
- net at C29.1: now also U4.24 (DREG)
- net at C34.2: now also U4.3 (VREF)
- net at C28.1: now also U3.24 (DREG)
- net at C31.2: now also U3.2 (AREG)
- net at R10.1, R9.1: now also U2.3 (FB)
- net at C32.2: now also U3.3 (VREF)
- net at L1.1: now also U2.8 (L1), U2.9 (L1)
- net at L1.2: now also U2.6 (L2), U2.7 (L2)
- net 3V45_D renamed 3V3_D
- net 3V3_D: now also R4.1, C50.2, U2.4 (VOUT), U2.5 (VOUT), U3.19 (IOVDD), U4.19 (IOVDD); no longer C14.2, C46.2, C47.2, U1.1 (IN), U1.3 (EN), U6.20 (DVDD)
- net To Test Point: no longer names the net of U6.7 (OUTR)
Other:
- moved on the sheet: R7, R8
