File: Onboard DSP Board HW/Main Board/MCU.kicad_sch (KiCad schematic)
At the start: 22 parts, among them U7 STM32H725RGVx, Y1 24.576MHz

Commit message: WIP
Parts:
- removed TP10: (no value), symbol Connector:TestPoint
- C100, C101, C102, C103, C2, C90, C91, C92, C93, C94, C95, C96, C97, C98, C99: footprint (none) -> Capacitor_SMD:C_0402_1005Metric
- L2: footprint (none) -> Inductor_SMD:L_Sunlord_SWPA252012S
- R14, R18: footprint (none) -> Resistor_SMD:R_0402_1005Metric
- U7: footprint (none) -> Package_DFN_QFN:QFN-68-1EP_8x8mm_P0.4mm_EP6.4x6.4mm

Commit message: WIP
Parts:
- removed C102: 100nF, Capacitor_SMD:C_0402_1005Metric, symbol Device:C
- removed C103: 1uF, Capacitor_SMD:C_0402_1005Metric, symbol Device:C
- removed Y1: 24.576MHz, symbol Device:Crystal
- added C104: 100nF, Capacitor_SMD:C_0402_1005Metric, symbol Device:C
- added C105: 4.7uF, Capacitor_SMD:C_0805_2012Metric, symbol Device:C
- added Y1: 24.576, Crystal:Crystal_SMD_3225-4Pin_3.2x2.5mm, symbol Device:Crystal_GND24
- C101: value 4.7uF -> 100nF
Connections:
- net 3V45_D: now also C104.1, C105.1
- net GND: now also C104.2, C105.2, Y1.2 (G), Y1.4 (G)
- net at C94.1, U7.11 (PH1): now also Y1.3
- net at C93.1, U7.10 (PH0): now also Y1.1

Commit message: WIP
Parts:
- Y1: value 24.576 -> 24Mhz; footprint Crystal:Crystal_SMD_3225-4Pin_3.2x2.5mm -> Crystal:Crystal_SMD_WE_IQXC-26-4Pin_1.6x1.2mm
Other:
- note removed: "HSE 24.576 MHz - integer-N PLL3 for 48k family"

Commit message: WIP
Connections:
- net BT1: no longer names the net of U7.36 (PB12)
- net BT2: no longer names the net of U7.39 (PB15)
- net USART3_CTS renamed UART3_CTS
- net USART3_RTS renamed UART3_RTS
- net USART3_RX renamed UART3_RX
- net USART3_TX renamed UART3_TX

Commit message: WIP
Connections:
- net LED: now also U7.32 (PB10); no longer U7.57 (PD2)
- net Pot2: now also U7.29 (PB0); no longer U7.14 (PC1)

Commit message: WIP
Parts:
- TP1: footprint (none) -> AWV:TestPoint_Plated_Hole_ID4_OD7.0mm

Commit message: WIP
Parts:
- added C102: 10uF, Capacitor_SMD:C_0603_1608Metric, symbol Device:C
- C93, C94: value 15pF -> 6.8pF
- C95: value 4.7uF -> 10uF; footprint Capacitor_SMD:C_0402_1005Metric -> Capacitor_SMD:C_0603_1608Metric
- L2: LCSC (none) -> C576403
- U7: LCSC (none) -> C5271073
- Y1: LCSC (none) -> C280834
Connections:
- net GND: now also C102.2
- net at C95.1, L2.1, U7.7 (VFBSMPS): now also C102.1
- net 3V45_D renamed 3V3_D
Other:
- note added: "SMPS direct (AN5419): 2.2uH VLX->VFB"
- note removed: "SMPS direct (AN5419): 2.2uH VLX->VFB, 4.7uF at VFB"
- moved on the sheet: C93, C94, Y1
