File: Onboard DSP Board HW/JFET String Preamp/untitled.kicad_sch (KiCad schematic)
At the start: 10 parts, among them J1 Input, Q1 MMBF201

Commit message: WIP
Parts:
- C3: value 100nF -> 100pF
Changed lines of the file:
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@@
 		)
 		(instances
-			(project "JFET String Preamp"
+			(project "JFET String Preamp Neck"
 				(path "/02ac84b2-5c3b-408e-9eb0-8fb87f64ec2b/0e773300-e149-4e84-baf2-886502bbe02a"
 					(reference "J12")
@@
 		)
 		(instances
-			(project "JFET String Preamp"
+			(project "JFET String Preamp Neck"
 				(path "/02ac84b2-5c3b-408e-9eb0-8fb87f64ec2b/0e773300-e149-4e84-baf2-886502bbe02a"
 					(reference "R7")
@@
 		)
 		(instances
-			(project "JFET String Preamp"
+			(project "JFET String Preamp Neck"
 				(path "/02ac84b2-5c3b-408e-9eb0-8fb87f64ec2b/0e773300-e149-4e84-baf2-886502bbe02a"
 					(reference "#PWR04")
@@
 		)
 		(instances
-			(project "JFET String Preamp"
+			(project "JFET String Preamp Neck"
 				(path "/02ac84b2-5c3b-408e-9eb0-8fb87f64ec2b/0e773300-e149-4e84-baf2-886502bbe02a"
 					(reference "R9")
@@
 		)
 		(instances
-			(project "JFET String Preamp"
+			(project "JFET String Preamp Neck"
 				(path "/02ac84b2-5c3b-408e-9eb0-8fb87f64ec2b/0e773300-e149-4e84-baf2-886502bbe02a"
 					(reference "J13")
@@
 		)
 		(instances
-			(project "JFET String Preamp"
+			(project "JFET String Preamp Neck"
 				(path "/02ac84b2-5c3b-408e-9eb0-8fb87f64ec2b/0e773300-e149-4e84-baf2-886502bbe02a"
 					(reference "J11")
@@
 		)
 		(instances
-			(project "JFET String Preamp"
+			(project "JFET String Preamp Neck"
 				(path "/02ac84b2-5c3b-408e-9eb0-8fb87f64ec2b/0e773300-e149-4e84-baf2-886502bbe02a"
 					(reference "C7")
@@
 		)
 		(instances
-			(project "JFET String Preamp"
+			(project "JFET String Preamp Neck"
 				(path "/02ac84b2-5c3b-408e-9eb0-8fb87f64ec2b/0e773300-e149-4e84-baf2-886502bbe02a"
 					(reference "R8")
@@
 			)
 		)
-		(property "Value" "100nF"
+		(property "Value" "100pF"
 			(at 80.518 68.834 0)
 			(show_name no)
@@
 		)
 		(instances
-			(project "JFET String Preamp"
+			(project "JFET String Preamp Neck"
 				(path "/02ac84b2-5c3b-408e-9eb0-8fb87f64ec2b/0e773300-e149-4e84-baf2-886502bbe02a"
 					(reference "C6")
@@
 		)
 		(instances
-			(project "JFET String Preamp"
+			(project "JFET String Preamp Neck"
 				(path "/02ac84b2-5c3b-408e-9eb0-8fb87f64ec2b/0e773300-e149-4e84-baf2-886502bbe02a"
 					(reference "J10")
@@
 		)
 		(instances
-			(project "JFET String Preamp"
+			(project "JFET String Preamp Neck"
 				(path "/02ac84b2-5c3b-408e-9eb0-8fb87f64ec2b/0e773300-e149-4e84-baf2-886502bbe02a"
 					(reference "Q3")
