File: Onboard DSP Board HW/JFET String Preamp/Neck Pickup/JFET String Preamp Neck.kicad_pcb (KiCad board)
At the start: 2 copper layers, 28.4 x 89.9 mm, 41 parts, among them J1 Input, J10 Input, J14 Input, J5 Input, Q1 MMBF201, Q2 MMBF201, Q3 MMBF201, Q4 MMBF201

Commit message: WIP
Parts:
- C3, C4, C6, C8: value 100nF -> 100pF

Commit message: WIP
Parts:
- Q1, Q2, Q3, Q4: value MMBF201 -> MMBFJ201
Routing:
- net GND: vias 32 -> 38
- net (no net): vias 3 -> 0
Other:
- board text added: "JLCJLCJLCJLC"
