File: Onboard DSP Board HW/OPA376 String Preamp/OPA376 String Preamp Bridge.kicad_pcb (KiCad board)
At the start: 2 copper layers, 28.4 x 92.7 mm, 48 parts, among them J1 Input, J10 Input, J14 Input, J5 Input, U1 TLV9001IDCK, U2 TLV9001IDCK, U3 TLV9001IDCK, U4 TLV9001IDCK

Commit message: WIP
Parts:
- J9: footprint Connector_JST:JST_SH_SM06B-SRSS-TB_1x06-1MP_P1.00mm_Horizontal -> Connector_PinHeader_2.00mm:PinHeader_1x06_P2.00mm_Horizontal
- moved J9 5.62 mm to (95.2, 56.0), turned to -90 degrees
- moved R1 4.12 mm to (107.4, 59.4), turned to -90 degrees
- moved C2 3.22 mm to (107.4, 57.4), turned to -90 degrees
- moved R2 3.20 mm to (106.5, 59.4), turned to 90 degrees
Connections:
- J9 pad 1: /SIngle FET preamp/3.3V -> GND
- J9 pad 2: /SIngle FET preamp/Output -> /SIngle FET preamp3/Output
- J9 pad 3: /SIngle FET preamp1/Output -> /SIngle FET preamp2/Output
- J9 pad 4: /SIngle FET preamp2/Output -> /SIngle FET preamp1/Output
- J9 pad 5: /SIngle FET preamp3/Output -> /SIngle FET preamp/Output
- J9 pad 6: GND -> /SIngle FET preamp/3.3V
Routing:
- net /SIngle FET preamp/MidRail: track 81.2 -> 77.5 mm
- net /SIngle FET preamp/3.3V: track 104.0 -> 101.3 mm, vias 5 -> 4
- net /SIngle FET preamp2/Output: track 58.5 -> 59.6 mm
- net /SIngle FET preamp3/Output: track 77.5 -> 78.2 mm
- net /SIngle FET preamp1/Output: track 40.5 -> 41.2 mm
Other:
- board text added: "V+"
