File: Onboard DSP Board HW/OPA376 String Preamp/untitled.kicad_sch (KiCad schematic)
At the start: 11 parts, among them J1 Input, U1 TLV9001IDCK

Commit message: WIP
Parts:
- C1: footprint Capacitor_SMD:C_0402_1005Metric -> Capacitor_SMD:C_0603_1608Metric
- U1: value TLV9001IDCK -> OPA376
Changed lines of the file:
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@@
 			)
 		)
-		(property "Value" "TLV9001IDCK"
+		(property "Value" "OPA376"
 			(at 183.134 72.136 0)
 			(show_name no)
@@
 			)
 		)
-		(property "Footprint" "Capacitor_SMD:C_0402_1005Metric"
+		(property "Footprint" "Capacitor_SMD:C_0603_1608Metric"
 			(at 149.86 52.07 0)
 			(hide yes)

Commit message: WIP
Parts:
- J1, J2, J3, J4: now left out of the parts list
Changed lines of the file:
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@@
 		(body_style 1)
 		(exclude_from_sim no)
-		(in_bom yes)
+		(in_bom no)
 		(on_board yes)
 		(in_pos_files yes)
@@
 		(body_style 1)
 		(exclude_from_sim no)
-		(in_bom yes)
+		(in_bom no)
 		(on_board yes)
 		(in_pos_files yes)
@@
 		(body_style 1)
 		(exclude_from_sim no)
-		(in_bom yes)
+		(in_bom no)
 		(on_board yes)
 		(in_pos_files yes)
@@
 		(body_style 1)
 		(exclude_from_sim no)
-		(in_bom yes)
-		(on_board yes)
-		(in_pos_files yes)
+		(in_bom no)
+		(on_board yes)
+		(in_pos_files yes)
