File: Onboard DSP Board HW/OPA376 String Preamp/OPA376 String Preamp.kicad_pcb (KiCad board)
At the start: 2 copper layers, 28.4 x 89.9 mm, 49 parts, among them J1 Input, J10 Input, J14 Input, J5 Input, U1 OPA376AIDCKT, U2 OPA376AIDCKT, U3 OPA376AIDCKT, U4 OPA376AIDCKT

Commit message: Add feedback caps damping resistors
Parts:
- removed C11, C13, C15: 22uF, Capacitor_SMD:C_0603_1608Metric
- removed C2: 10uF, Capacitor_SMD:C_0603_1608Metric
- added C3: 100nF, Capacitor_SMD:C_0603_1608Metric, F.Cu at (107.7, 64.6)
- added U5: OPA376AIDCKT, Package_TO_SOT_SMD:SOT-353_SC-70-5, F.Cu at (101.3, 100.0)
- C1: value 22uF -> 47uF; footprint Capacitor_SMD:C_0603_1608Metric -> Capacitor_Tantalum_SMD:CP_EIA-3216-18_Kemet-A
- moved C1 24.8 mm to (95.0, 99.8), turned to 180 degrees
- moved R2 4.50 mm to (98.2, 100.0)
- moved R1 2.45 mm to (99.2, 100.0)
- moved R3 0.35 mm to (107.7, 61.2), turned to -90 degrees
Connections:
- net /Input renamed Net-(J1-Pin_1)
- net /SIngle FET preamp1/Input renamed Net-(J5-Pin_1)
- net /SIngle FET preamp2/Input renamed Net-(J10-Pin_1)
- net /SIngle FET preamp3/Input renamed Net-(J14-Pin_1)
- C1 pad 1: GND -> Net-(U5-+)
- C1 pad 2: Net-(C1-Pad2) -> GND
- J9 pad 6: Net-(J9-Pin_6) -> /3V3
- R1 pad 2: /SIngle FET preamp/MidRail -> Net-(U5-+)
- R14 pad 1: Net-(C1-Pad2) -> /SIngle FET preamp/MidRail
- R17 pad 1: Net-(C11-Pad2) -> /SIngle FET preamp/MidRail
- R2 pad 1: /SIngle FET preamp/MidRail -> Net-(U5-+)
- R20 pad 1: Net-(C13-Pad2) -> /SIngle FET preamp/MidRail
- R23 pad 1: Net-(C15-Pad2) -> /SIngle FET preamp/MidRail
- R3 pad 1: /SIngle FET preamp/3.3V -> /3V3
- R3 pad 2: Net-(J9-Pin_6) -> /SIngle FET preamp/3.3V
Routing:
- net /SIngle FET preamp/MidRail: track 82.0 -> 120.9 mm, vias 0 -> 8
- net Net-(U5-+): track 0.00 -> 4.44 mm
- net /3V3: track 0.00 -> 4.04 mm
- net Net-(J9-Pin_6): track 3.69 -> 0.00 mm
- net /SIngle FET preamp/3.3V: track 82.5 -> 85.9 mm, vias 5 -> 6
- net Net-(C15-Pad2): track 1.70 -> 0.00 mm
- net Net-(C13-Pad2): track 1.68 -> 0.00 mm
- net Net-(C11-Pad2): track 1.62 -> 0.00 mm
- net Net-(C1-Pad2): track 1.40 -> 0.00 mm
- net GND: track 9.63 -> 10.8 mm, vias 24 -> 28

Commit message: WIP
Parts:
- added C11: 220pF, Capacitor_SMD:C_0402_1005Metric, F.Cu at (100.8, 76.3)
- added C13: 220pF, Capacitor_SMD:C_0402_1005Metric, F.Cu at (100.8, 93.8)
- added C15: 220pF, Capacitor_SMD:C_0402_1005Metric, F.Cu at (101.0, 111.2)
- added C21: 220pF, Capacitor_SMD:C_0402_1005Metric, F.Cu at (101.5, 128.5)
- added R25: 15k, Resistor_SMD:R_0402_1005Metric, F.Cu at (97.4, 74.0)
- added R26: 15k, Resistor_SMD:R_0402_1005Metric, F.Cu at (97.5, 91.4)
- added R27: 15k, Resistor_SMD:R_0402_1005Metric, F.Cu at (97.4, 108.8)
- added R28: 15k, Resistor_SMD:R_0402_1005Metric, F.Cu at (97.5, 126.1)
- C1: footprint Capacitor_Tantalum_SMD:CP_EIA-3216-18_Kemet-A -> Capacitor_Tantalum_SMD:CP_EIA-3216-12_Kemet-S
Connections:
- net Net-(J1-Pin_1) renamed /SIngle FET preamp/in
- net Net-(J10-Pin_1) renamed /SIngle FET preamp2/in
- net Net-(J14-Pin_1) renamed /SIngle FET preamp3/in
- net Net-(J5-Pin_1) renamed /SIngle FET preamp1/in
Routing:
- net Net-(U2--): track 2.33 -> 3.64 mm
- net /SIngle FET preamp1/Output: track 39.4 -> 40.7 mm
- net /SIngle FET preamp2/Output: track 56.9 -> 58.2 mm
- net Net-(U3--): track 2.33 -> 3.54 mm
- net Net-(U4--): track 2.33 -> 3.52 mm
- net /SIngle FET preamp/Output: track 20.9 -> 22.1 mm
- net /SIngle FET preamp3/Output: track 74.7 -> 75.9 mm
- net Net-(U1--): track 2.33 -> 3.47 mm
- net Net-(U3-+): track 2.16 -> 3.26 mm
- net Net-(U1-+): track 2.16 -> 3.26 mm
- net Net-(U2-+): track 2.16 -> 3.24 mm
- net Net-(U4-+): track 2.16 -> 3.24 mm

Commit message: preamp board modified and simulated
Parts:
- removed J9: ~, Connector_PinHeader_2.00mm:PinHeader_1x06_P2.00mm_Horizontal
- removed R1: 100K, Resistor_SMD:R_0402_1005Metric
- added J18: Conn_01x07_Pin, Connector_PinHeader_2.00mm:PinHeader_1x07_P2.00mm_Horizontal, B.Cu at (93.8, 57.7)
- C1: value 47uF -> 100pF; footprint Capacitor_Tantalum_SMD:CP_EIA-3216-12_Kemet-S -> Capacitor_SMD:C_0402_1005Metric
- R2: value 43K -> 1K
- R25, R26, R27, R28: value 15k -> 27K
- moved C1 4.21 mm to (99.2, 99.6), turned to -90 degrees
- moved R2 0.38 mm to (98.0, 99.6), turned to 90 degrees
Connections:
- R2 pad 1: Net-(U5-+) -> /Bias
- R2 pad 2: GND -> Net-(U5-+)
- R25 pad 1: GND -> /SIngle FET preamp/MidRail
- R26 pad 1: GND -> /SIngle FET preamp/MidRail
- R27 pad 1: GND -> /SIngle FET preamp/MidRail
- R28 pad 1: GND -> /SIngle FET preamp/MidRail
Routing:
- net /Bias: track 0.00 -> 49.2 mm, vias 0 -> 1
- net /SIngle FET preamp/MidRail: track 121.1 -> 131.5 mm
- net /SIngle FET preamp/3.3V: track 85.9 -> 80.8 mm, vias 6 -> 5
- net Net-(U5-+): track 4.44 -> 2.55 mm
- net GND: track 10.8 -> 12.4 mm, vias 28 -> 33
- net /3V3: track 4.04 -> 3.42 mm

Commit message: WIP
Parts:
- J18: value Conn_01x07_Pin -> ~
- U1, U2, U3, U4, U5: value OPA376AIDCKT -> OPA376AIDCKR
Connections:
- J18 pad 3: /SIngle FET preamp3/Output -> /3V3
- J18 pad 4: /SIngle FET preamp2/Output -> /SIngle FET preamp3/Output
- J18 pad 5: /SIngle FET preamp1/Output -> /SIngle FET preamp2/Output
- J18 pad 6: /SIngle FET preamp/Output -> /SIngle FET preamp1/Output
- J18 pad 7: /3V3 -> /SIngle FET preamp/Output
Routing:
- net /3V3: track 3.42 -> 10.9 mm
- net /SIngle FET preamp1/Output: track 40.9 -> 40.1 mm
- net /SIngle FET preamp3/Output: track 76.1 -> 75.3 mm
- net /SIngle FET preamp2/Output: track 58.4 -> 57.6 mm
- net GND: vias 33 -> 32

Commit message: WIP
Parts:
- moved C16 1.34 mm to (97.5, 126.4)
- moved C17 1.34 mm to (100.6, 70.6)
- moved C21 1.34 mm to (101.4, 129.8)
- moved J1 1.34 mm to (93.4, 67.5)
- moved J14 1.34 mm to (93.4, 122.2)
- moved J16 1.34 mm to (106.6, 122.2)
- moved J2 1.34 mm to (106.6, 77.8)
- moved J3 1.34 mm to (93.4, 77.8)
- moved J4 1.34 mm to (106.6, 67.5)
- moved R22 1.34 mm to (97.5, 125.4)
- moved R28 1.34 mm to (97.4, 127.4)
- moved U1 1.34 mm to (100.0, 72.3)
- moved C10 1.34 mm to (97.5, 71.7)
- moved C11 1.34 mm to (100.8, 75.0)
- moved C20 1.34 mm to (100.6, 125.3)
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Routing:
- net /SIngle FET preamp/MidRail: track 131.5 -> 135.1 mm
- net /SIngle FET preamp2/Output: track 57.6 -> 59.4 mm
- net /SIngle FET preamp/Output: track 22.5 -> 21.0 mm
- net /SIngle FET preamp3/Output: track 75.3 -> 76.6 mm
- net /SIngle FET preamp/3.3V: track 80.8 -> 81.7 mm
- net /SIngle FET preamp1/Output: track 40.1 -> 39.5 mm
Other:
- board size 28.4 x 89.9 mm -> 28.4 x 92.7 mm
