File: Onboard DSP Board HW/String Preamp Test Board/charger.kicad_sch (KiCad schematic)
At the start: 12 parts, among them J1 Battery, J4 Output Jack, U1 TLV9002, U2 TP4054

Commit message: WIP
Parts:
- renumbered C5 to C12, C6 to C13, C8 to C14, C9 to C15, J1 to J3, R1 to R24, R2 to R25, R7 to R26, U1 to U4, U2 to U5
Changed lines of the file:
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@@
 		(dnp no)
 		(fields_autoplaced yes)
-		(property "Reference" "R1"
+		(property "Reference" "R24"
 			(at 118.11 92.7099 0)
 			(show_name no)
@@
 			(project "String Preamp Test Board"
 				(path "/17071b06-4887-4c2e-9588-4148705cb0ef/d43362dd-6fda-43c9-aeea-4941a9e2c436"
-					(reference "R1")
+					(reference "R24")
 					(unit 1)
 				)
@@
 		(dnp no)
 		(fields_autoplaced yes)
-		(property "Reference" "C6"
+		(property "Reference" "C13"
 			(at 129.54 106.6799 0)
 			(show_name no)
@@
 			(project "String Preamp Test Board"
 				(path "/17071b06-4887-4c2e-9588-4148705cb0ef/d43362dd-6fda-43c9-aeea-4941a9e2c436"
-					(reference "C6")
+					(reference "C13")
 					(unit 1)
 				)
@@
 		(in_pos_files yes)
 		(dnp no)
-		(property "Reference" "C5"
+		(property "Reference" "C12"
 			(at 119.38 67.31 0)
 			(show_name no)
@@
 			(project "String Preamp Test Board"
 				(path "/17071b06-4887-4c2e-9588-4148705cb0ef/d43362dd-6fda-43c9-aeea-4941a9e2c436"
-					(reference "C5")
+					(reference "C12")
 					(unit 1)
 				)
@@
 		(in_pos_files yes)
 		(dnp no)
-		(property "Reference" "#PWR04"
+		(property "Reference" "#PWR019"
 			(at 105.41 123.19 0)
 			(hide yes)
@@
 			(project "String Preamp Test Board"
 				(path "/17071b06-4887-4c2e-9588-4148705cb0ef/d43362dd-6fda-43c9-aeea-4941a9e2c436"
-					(reference "#PWR04")
+					(reference "#PWR019")
 					(unit 1)
 				)
@@
 		(in_pos_files yes)
 		(dnp no)
-		(property "Reference" "U2"
+		(property "Reference" "U5"
 			(at 140.2206 57.2602 0)
 			(show_name no)
@@
 			(project "String Preamp Test Board"
 				(path "/17071b06-4887-4c2e-9588-4148705cb0ef/d43362dd-6fda-43c9-aeea-4941a9e2c436"
-					(reference "U2")
+					(reference "U5")
 					(unit 1)
 				)
@@
 		(in_pos_files yes)
 		(dnp no)
-		(property "Reference" "R7"
+		(property "Reference" "R26"
 			(at 153.67 71.12 90)
 			(show_name no)
@@
 			(project "String Preamp Test Board"
 				(path "/17071b06-4887-4c2e-9588-4148705cb0ef/d43362dd-6fda-43c9-aeea-4941a9e2c436"
-					(reference "R7")
+					(reference "R26")
 					(unit 1)
 				)
@@
 		(dnp no)
 		(fields_autoplaced yes)
-		(property "Reference" "C9"
+		(property "Reference" "C15"
 			(at 162.56 58.4199 0)
 			(show_name no)
@@
 			(project "String Preamp Test Board"
 				(path "/17071b06-4887-4c2e-9588-4148705cb0ef/d43362dd-6fda-43c9-aeea-4941a9e2c436"
-					(reference "C9")
+					(reference "C15")
 					(unit 1)
 				)
@@
 		(in_pos_files yes)
 		(dnp no)
-		(property "Reference" "U1"
+		(property "Reference" "U4"
 			(at 104.14 101.6001 0)
 			(show_name no)
@@
 			(project "String Preamp Test Board"
 				(path "/17071b06-4887-4c2e-9588-4148705cb0ef/d43362dd-6fda-43c9-aeea-4941a9e2c436"
-					(reference "U1")
+					(reference "U4")
 					(unit 3)
 				)
@@
 		(dnp no)
 		(fields_autoplaced yes)
-		(property "Reference" "#PWR08"
+		(property "Reference" "#PWR021"
 			(at 193.04 77.47 0)
 			(hide yes)
@@
 			(project "String Preamp Test Board"
 				(path "/17071b06-4887-4c2e-9588-4148705cb0ef/d43362dd-6fda-43c9-aeea-4941a9e2c436"
-					(reference "#PWR08")
+					(reference "#PWR021")
 					(unit 1)
 				)
@@
 		(in_pos_files yes)
 		(dnp no)
-		(property "Reference" "J1"
+		(property "Reference" "J3"
 			(at 84.455 87.596 0)
 			(show_name no)
@@
 			(project "String Preamp Test Board"
 				(path "/17071b06-4887-4c2e-9588-4148705cb0ef/d43362dd-6fda-43c9-aeea-4941a9e2c436"
-					(reference "J1")
+					(reference "J3")
 					(unit 1)
 				)
@@
 		(dnp no)
 		(fields_autoplaced yes)
-		(property "Reference" "#PWR07"
+		(property "Reference" "#PWR020"
 			(at 139.7 85.09 0)
 			(hide yes)
@@
 			(project "String Preamp Test Board"
 				(path "/17071b06-4887-4c2e-9588-4148705cb0ef/d43362dd-6fda-43c9-aeea-4941a9e2c436"
-					(reference "#PWR07")
+					(reference "#PWR020")
 					(unit 1)
 				)
@@
 		(dnp no)
 		(fields_autoplaced yes)
-		(property "Reference" "C8"
+		(property "Reference" "C14"
 			(at 142.621 98.2253 0)
 			(show_name no)
@@
 			(project "String Preamp Test Board"
 				(path "/17071b06-4887-4c2e-9588-4148705cb0ef/d43362dd-6fda-43c9-aeea-4941a9e2c436"
-					(reference "C8")
+					(reference "C14")
 					(unit 1)
 				)
@@
 		(dnp no)
 		(fields_autoplaced yes)
-		(property "Reference" "R2"
+		(property "Reference" "R25"
 			(at 118.11 106.6799 0)
 			(show_name no)
@@
 			(project "String Preamp Test Board"
 				(path "/17071b06-4887-4c2e-9588-4148705cb0ef/d43362dd-6fda-43c9-aeea-4941a9e2c436"
-					(reference "R2")
+					(reference "R25")
 					(unit 1)
 				)
