File: Onboard DSP Board HW/String Preamp Test Board/String Preamp Test Board.kicad_sch (KiCad schematic)
At the start: 24 parts, among them U1 TLV9004

Commit message: move bias to cavity
Parts:
- added R14: 9.6k, symbol Device:R
- added R15: 2.2k, symbol Device:R
- C2, C3: value 8.2nF -> 5.6nF
- R3: value 10K -> 14.7k
- R4: value 10K -> 5.9K
Connections:
- net VG: now also R14.1
- net at C2.1, R3.2, R4.1: now also R14.2
- net filt_in: no longer names the net of C2.2, R6.2, U1.8
- net filt_in: now also R15.1; no longer R27.1, RV2.2
- new net filt_out: R15.2, R27.1, RV2.2
Other:
- moved on the sheet: C2, C3, C6, R3, R4, RV2, U1C
