File: Onboard DSP Board HW/String Preamp Test Board/String Preamp Test Board.kicad_sch (KiCad schematic)
At the start: 32 parts, among them J3 Battery, J4 Output Jack, U1 TLV9004, U5 TP4054

Commit message: WIP
Parts:
- C13, C14: value 0.1uF -> 100nF
- C6: value 4.7nF -> 5.6nF
- C7: footprint Capacitor_SMD:C_1206_3216Metric -> Capacitor_Tantalum_SMD:CP_EIA-3216-10_Kemet-I
- R14: value 9.6k -> 10K
- R3: value 14.7k -> 15K
- R4: value 5.9K -> 6.2K
- R6: value 15k -> 15K
- RV3: value (none) -> 10K
- U1: footprint Package_SO:TSSOP-14_4.4x3.6mm_P0.4mm -> Package_SO:SOIC-14_3.9x8.7mm_P1.27mm
Connections:
- net GND: now also U1.11 (V-); no longer U1.4 (V+)
- net buf_in: now also U1.10 (+); no longer U1.5 (+)
- net filt_out: now also RV2.1
- net v+: now also U1.4 (V+); no longer U1.11 (V-)
- net at C2.2, R15.1, R6.2: now also U1.7; no longer U1.8
- net at C3.1, R4.2: now also U1.5 (+); no longer U1.10 (+)
- net at R5.2, R6.1: now also U1.6 (-); no longer U1.9 (-)
- new net: R9.1, U1.8, U1.9 (-)
Other:
- moved on the sheet: RV2
Changed lines of the file:
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@@
 	)
 	(junction
+		(at 210.82 109.22)
+		(diameter 0)
+		(color 0 0 0 0)
+	)
+	(junction
+		(at 193.04 115.57)
+		(diameter 0)
+		(color 0 0 0 0)
+	)
+	(junction
 		(at 50.8 102.87)
 		(diameter 0)
@@
 	)
 	(junction
-		(at 210.82 109.22)
-		(diameter 0)
-		(color 0 0 0 0)
-	)
-	(junction
 		(at 128.27 67.31)
 		(diameter 0)
@@
 	(wire
 		(pts
+			(xy 198.12 109.22) (xy 193.04 109.22)
+		)
+		(stroke
+			(width 0)
+			(type default)
+		)
+	)
+	(wire
+		(pts
 			(xy 198.12 34.29) (xy 195.58 34.29)
 		)
@@
 	(wire
 		(pts
-			(xy 204.47 109.22) (xy 210.82 109.22)
+			(xy 205.74 109.22) (xy 210.82 109.22)
 		)
 		(stroke
@@
 	(wire
 		(pts
-			(xy 200.66 113.03) (xy 200.66 115.57)
+			(xy 193.04 115.57) (xy 201.93 115.57)
+		)
+		(stroke
+			(width 0)
+			(type default)
+		)
+	)
+	(wire
+		(pts
+			(xy 201.93 113.03) (xy 201.93 115.57)
 		)
 		(stroke
@@
 	(wire
 		(pts
-			(xy 190.5 115.57) (xy 200.66 115.57)
+			(xy 190.5 115.57) (xy 193.04 115.57)
 		)
 		(stroke
@@
 	(wire
 		(pts
+			(xy 193.04 109.22) (xy 193.04 115.57)
+		)
+		(stroke
+			(width 0)
+			(type default)
+		)
+	)
+	(wire
+		(pts
 			(xy 137.16 116.84) (xy 137.16 120.65)
 		)
@@
 	)
 	(label "filt_out"
-		(at 191.77 115.57 0)
+		(at 194.31 115.57 0)
 		(effects
 			(font
@@
 			)
 		)
-		(property "Footprint" "Package_SO:TSSOP-14_4.4x3.6mm_P0.4mm"
+		(property "Footprint" "Package_SO:SOIC-14_3.9x8.7mm_P1.27mm"
 			(at 146.05 64.77 0)
 			(hide yes)
@@
 			)
 		)
-		(property "Value" ""
+		(property "Value" "10K"
 			(at 109.22 46.99 0)
 			(show_name no)
@@
 		(at 223.52 106.68 0)
 		(mirror x)
-		(unit 2)
+		(unit 3)
 		(body_style 1)
 		(exclude_from_sim no)
@@
 			)
 		)
-		(property "Footprint" "Package_SO:TSSOP-14_4.4x3.6mm_P0.4mm"
+		(property "Footprint" "Package_SO:SOIC-14_3.9x8.7mm_P1.27mm"
 			(at 223.52 106.68 0)
 			(hide yes)
@@
 				(path "/17071b06-4887-4c2e-9588-4148705cb0ef"
 					(reference "U1")
-					(unit 2)
+					(unit 3)
 				)
 			)
@@
 			)
 		)
-		(property "Value" "0.1uF"
+		(property "Value" "100nF"
 			(at 193.421 66.4722 0)
 			(show_name no)
@@
 		(unit 1)
 		(body_style 1)
-		(exclude_from_sim no)
+		(exclude_from_sim yes)
 		(in_bom yes)
 		(on_board yes)
@@
 		(unit 1)
 		(body_style 1)
-		(exclude_from_sim no)
+		(exclude_from_sim yes)
 		(in_bom yes)
 		(on_board yes)
@@
 		)
 		(property "Value" "Battery"
-			(at 62.23 43.18 0)
+			(at 76.2 48.26 0)
 			(show_name no)
 			(do_not_autoplace no)
@@
 		(dnp no)
 		(property "Reference" "RV3"
-			(at 259.08 114.3001 0)
+			(at 258.572 113.538 0)
 			(show_name no)
 			(do_not_autoplace no)
@@
 			)
 		)
-		(property "Value" ""
-			(at 261.62 114.3 0)
+		(property "Value" "10K"
+			(at 256.286 116.078 0)
 			(show_name no)
 			(do_not_autoplace no)
@@
 			)
 		)
-		(property "Footprint" "Package_SO:TSSOP-14_4.4x3.6mm_P0.4mm"
+		(property "Footprint" "Package_SO:SOIC-14_3.9x8.7mm_P1.27mm"
 			(at 106.68 116.84 0)
 			(hide yes)
@@
 		(unit 1)
 		(body_style 1)
-		(exclude_from_sim no)
+		(exclude_from_sim yes)
 		(in_bom yes)
 		(on_board yes)
@@
 		(unit 1)
 		(body_style 1)
-		(exclude_from_sim no)
+		(exclude_from_sim yes)
 		(in_bom yes)
 		(on_board yes)
@@
 			)
 		)
-		(property "Value" "4.7nF"
+		(property "Value" "5.6nF"
 			(at 214.63 115.5699 0)
 			(show_name no)
@@
 			)
 		)
-		(property "Value" "0.1uF"
+		(property "Value" "100nF"
 			(at 132.08 74.9299 0)
 			(show_name no)
@@
 			)
 		)
-		(property "Value" "5.9K"
+		(property "Value" "6.2K"
 			(at 149.86 113.03 90)
 			(show_name no)
@@
 			)
 		)
-		(property "Value" "14.7k"
+		(property "Value" "15K"
 			(at 129.54 113.03 90)
 			(show_name no)
@@
 			)
 		)
-		(property "Value" "15k"
+		(property "Value" "15K"
 			(at 168.91 96.52 90)
 			(show_name no)
@@
 			)
 		)
-		(property "Value" "9.6k"
-			(at 130.81 125.476 0)
+		(property "Value" "10K"
+			(at 129.794 125.476 0)
 			(show_name no)
 			(do_not_autoplace no)
 			(effects
 				(font
+					(face "SF Compact")
 					(size 1.27 1.27)
 				)
@@
 	(symbol
 		(lib_id "Device:R_Potentiometer")
-		(at 200.66 109.22 90)
+		(at 201.93 109.22 90)
 		(mirror x)
 		(unit 1)
@@
 		(dnp no)
 		(property "Reference" "RV2"
-			(at 200.66 102.87 90)
+			(at 201.93 102.87 90)
 			(show_name no)
 			(do_not_autoplace no)
@@
 		)
 		(property "Value" "A100K"
-			(at 200.66 105.41 90)
+			(at 201.93 105.41 90)
 			(show_name no)
 			(do_not_autoplace no)
@@
 		)
 		(property "Footprint" "Potentiometer_THT:Potentiometer_Alps_RK097_Single_Horizontal"
-			(at 200.66 109.22 0)
+			(at 201.93 109.22 0)
 			(hide yes)
 			(show_name no)
@@
 		)
 		(property "Datasheet" ""
-			(at 200.66 109.22 0)
+			(at 201.93 109.22 0)
 			(hide yes)
 			(show_name no)
@@
 		)
 		(property "Description" "Potentiometer"
-			(at 200.66 109.22 0)
+			(at 201.93 109.22 0)
 			(hide yes)
 			(show_name no)
@@
 		)
 		(property "Sim.Device" "R"
-			(at 200.66 109.22 0)
+			(at 201.93 109.22 0)
 			(hide yes)
 			(show_name no)
@@
 		)
 		(property "Sim.Type" "POT"
-			(at 200.66 109.22 0)
+			(at 201.93 109.22 0)
 			(hide yes)
 			(show_name no)
@@
 		)
 		(property "Sim.Pins" "1=r0 2=wiper 3=r1"
-			(at 200.66 109.22 0)
+			(at 201.93 109.22 0)
 			(hide yes)
 			(show_name no)
@@
 		(lib_id "Amplifier_Operational:Opamp_Quad")
 		(at 176.53 64.77 0)
-		(mirror x)
 		(unit 5)
 		(body_style 1)
@@
 		(dnp no)
 		(property "Reference" "U1"
-			(at 178.054 59.944 0)
+			(at 178.054 69.596 0)
 			(show_name no)
 			(do_not_autoplace no)
@@
 		)
 		(property "Value" "TLV9004"
-			(at 179.832 70.104 0)
+			(at 179.832 59.436 0)
 			(show_name no)
 			(do_not_autoplace no)
@@
 			)
 		)
-		(property "Footprint" "Package_SO:TSSOP-14_4.4x3.6mm_P0.4mm"
+		(property "Footprint" "Package_SO:SOIC-14_3.9x8.7mm_P1.27mm"
 			(at 176.53 64.77 0)
 			(hide yes)
@@
 		)
 		(property "Description" "Quad operational amplifier"
-			(at 176.53 55.88 0)
+			(at 176.53 73.66 0)
 			(hide yes)
 			(show_name no)
@@
 		)
 		(property "Sim.Library" "tlv9004.lib"
-			(at 163.83 52.07 0)
+			(at 163.83 77.47 0)
 			(hide yes)
 			(show_name yes)
@@
 		)
 		(property "Sim.Name" "TLV9004"
-			(at 163.83 44.45 0)
+			(at 163.83 85.09 0)
 			(hide yes)
 			(show_name yes)
@@
 		)
 		(property "Sim.Device" "SUBCKT"
-			(at 163.83 46.99 0)
+			(at 163.83 82.55 0)
 			(hide yes)
 			(show_name yes)
@@
 		)
 		(property "Sim.Pins" "1=OUT1 2=IN1- 3=IN1+ 4=VCC 5=IN2+ 6=IN2- 7=OUT2 8=OUT3 9=IN3- 10=IN3+ 11=VEE 12=IN4+ 13=IN4- 14=OUT4"
-			(at 163.83 49.53 0)
+			(at 163.83 80.01 0)
 			(hide yes)
 			(show_name yes)
@@
 		)
 		(property private "KLC_S3.1" "Units A+B are centered, UnitC has a offset so it fits nicely on A or B."
-			(at 163.83 40.64 0)
+			(at 163.83 88.9 0)
 			(hide yes)
 			(show_name yes)
@@
 		)
 		(property private "KLC_S4.1" "Pin1 and Pin7 are the output, adding a name would look ugly and does not add a benefit."
-			(at 163.83 38.1 0)
+			(at 163.83 91.44 0)
 			(hide yes)
 			(show_name yes)
@@
 		)
 		(property private "KLC_S6.2" "This is a generic symbol and thus has no datasheet."
-			(at 163.83 35.56 0)
+			(at 163.83 93.98 0)
 			(hide yes)
 			(show_name yes)
@@
 		(unit 1)
 		(body_style 1)
-		(exclude_from_sim no)
+		(exclude_from_sim yes)
 		(in_bom yes)
 		(on_board yes)
@@
 		(unit 1)
 		(body_style 1)
-		(exclude_from_sim no)
+		(exclude_from_sim yes)
 		(in_bom no)
 		(on_board yes)
@@
 		(at 168.91 114.3 0)
 		(mirror x)
-		(unit 3)
+		(unit 2)
 		(body_style 1)
 		(exclude_from_sim no)
@@
 			)
 		)
-		(property "Footprint" "Package_SO:TSSOP-14_4.4x3.6mm_P0.4mm"
+		(property "Footprint" "Package_SO:SOIC-14_3.9x8.7mm_P1.27mm"
 			(at 168.91 114.3 0)
 			(hide yes)
@@
 				(path "/17071b06-4887-4c2e-9588-4148705cb0ef"
 					(reference "U1")
-					(unit 3)
+					(unit 2)
 				)
 			)
@@
 			)
 		)
-		(property "Footprint" "Capacitor_SMD:C_1206_3216Metric"
+		(property "Footprint" "Capacitor_Tantalum_SMD:CP_EIA-3216-10_Kemet-I"
 			(at 254 105.7148 0)
 			(hide yes)
