File: Onboard DSP Board HW/String Preamp Test Board/String Preamp Test Board.kicad_pcb (KiCad board)
At the start: 2 copper layers, 85.9 x 24.5 mm, 51 parts, among them J1 Conn_01x07_Socket, J2 Conn_01x07_Socket, J3 Battery, J4 Output Jack, U1 TLV9004, U2 TLV9001IDCK, U3 TLV9001IDCK, U5 TP4054

Commit message: WIP
Parts:
- C13, C14: value 0.1uF -> 100nF
- C6: value 4.7nF -> 5.6nF
- C7: footprint Capacitor_SMD:C_1206_3216Metric -> Capacitor_Tantalum_SMD:CP_EIA-3216-10_Kemet-I
- R14: value 9.6k -> 10K
- R3: value 14.7k -> 15K
- R4: value 5.9K -> 6.2K
- R6: value 15k -> 15K
- RV10, RV11, RV4, RV5, RV6, RV7, RV8, RV9: footprint Potentiometer_SMD:Potentiometer_Bourns_TC33X_Vertical -> TC33X_Local:Potentiometer_Bourns_TC33X_Vertical_HandSolder
- RV3: value ~ -> 10K
- U1: footprint Package_SO:TSSOP-14_4.4x3.6mm_P0.4mm -> Package_SO:SOIC-14_3.9x8.7mm_P1.27mm
- moved C14 11.0 mm to (120.2, 63.4)
- moved R25 6.82 mm to (123.7, 71.8), turned to 180 degrees
- moved C13 6.32 mm to (123.7, 68.4), turned to 180 degrees
- moved C2 5.01 mm to (116.3, 60.2)
- moved C3 5.01 mm to (121.9, 60.3)
- moved R14 5.01 mm to (119.1, 59.0)
- moved R3 5.01 mm to (119.1, 60.3)
- moved R5 5.01 mm to (113.8, 59.0)
- moved R6 5.01 mm to (113.8, 60.3)
- moved R15 5.01 mm to (113.8, 61.6)
- moved R4 5.01 mm to (119.1, 61.6)
- moved R24 4.97 mm to (123.7, 70.1), turned to 0 degrees
- moved U1 3.77 mm to (116.9, 68.2), turned to -90 degrees
- moved R9 3.20 mm to (125.2, 64.5)
- moved J1 0.55 mm to (75.0, 65.2)
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Connections:
- C3 pad 1: Net-(U1C-+) -> Net-(U1B-+)
- R4 pad 2: Net-(U1C-+) -> Net-(U1B-+)
- R5 pad 2: Net-(U1C--) -> Net-(U1B--)
- R6 pad 1: Net-(U1C--) -> Net-(U1B--)
- R9 pad 1: Net-(U1B--) -> Net-(U1C--)
- RV10 pad 1: GND -> /VG
- RV11 pad 1: GND -> /VG
- RV2 pad 1: unconnected-(RV2-Pad1) -> /filt_out
- RV4 pad 1: GND -> /VG
- RV5 pad 1: GND -> /VG
- RV6 pad 1: GND -> /VG
- RV7 pad 1: GND -> /VG
- RV8 pad 1: GND -> /VG
- RV9 pad 1: GND -> /VG
- U1 pad 10: Net-(U1C-+) -> /buf_in
- U1 pad 11: /v+ -> GND
- U1 pad 4: GND -> /v+
- U1 pad 5: /buf_in -> Net-(U1B-+)
- U1 pad 7: Net-(U1B--) -> Net-(C2-Pad2)
- U1 pad 8: Net-(C2-Pad2) -> Net-(U1C--)
Routing:
- net /VG: track 85.8 -> 141.1 mm, vias 4 -> 5
- net /buf_in: track 60.4 -> 47.7 mm
- net Net-(U1D-+): track 21.8 -> 10.9 mm
- net Net-(U1B-+): track 0.00 -> 8.58 mm
- net GND: track 16.9 -> 8.41 mm
- net Net-(U1C-+): track 7.96 -> 0.00 mm
- net /v+: track 114.1 -> 121.2 mm
- net Net-(U1B--): track 2.12 -> 8.87 mm, vias 0 -> 2
- net /filt_out: track 53.8 -> 59.1 mm
- net /sum_in: track 21.4 -> 16.8 mm, vias 1 -> 0
- net Net-(C2-Pad2): track 10.4 -> 8.67 mm
- net /sum_out: track 12.7 -> 10.9 mm
- net Net-(U1C--): track 13.2 -> 14.7 mm, vias 2 -> 0
- net Net-(C7-Pad1): track 15.3 -> 13.8 mm
- net Net-(J2-Pin_6): track 3.96 -> 4.86 mm
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
Commit message: WIP
Parts:
- moved C11 0.55 mm to (98.7, 77.4)
- moved C6 0.55 mm to (83.7, 78.4)
- moved R11 0.55 mm to (83.0, 74.4)
- moved R12 0.55 mm to (79.1, 74.4)
- moved R16 0.55 mm to (87.3, 75.9)
- moved R17 0.55 mm to (103.8, 74.2)
- moved C9 0.55 mm to (91.4, 77.2)
- moved R10 0.55 mm to (86.8, 74.3)
- moved R13 0.55 mm to (75.7, 74.3)
- moved R18 0.55 mm to (99.9, 74.2)
- moved R19 0.55 mm to (96.0, 74.2)
- moved R2 0.55 mm to (103.6, 76.3)
- moved R20 0.55 mm to (92.8, 74.2)
- moved R23 0.55 mm to (94.6, 76.6)
- moved RV10 0.55 mm to (96.0, 70.7)
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Routing:
- net /VG: track 141.1 -> 142.2 mm
- net /filt_out: track 59.1 -> 58.1 mm
- net /v+: track 121.2 -> 122.3 mm
- net Net-(J1-Pin_7): track 3.56 -> 4.11 mm
- net /p1_out: track 35.8 -> 35.3 mm
Other:
- rule pad_to_mask_clearance: 0 -> 0.05
