File: Onboard DSP Board HW/String Preamp Test Board/Summer.kicad_sch (KiCad schematic)
At the start: 13 parts, among them J1 Conn_01x07_Socket, U2 TLV9001IDCK

Commit message: WIP
Parts:
- RV4, RV5, RV6, RV7: footprint Potentiometer_SMD:Potentiometer_Bourns_TC33X_Vertical -> TC33X_Local:Potentiometer_Bourns_TC33X_Vertical_HandSolder
Connections:
- net GND: no longer RV4.1, RV5.1, RV6.1, RV7.1
- net VG: now also RV4.1, RV5.1, RV6.1, RV7.1
Other:
- moved on the sheet: J1

Commit message: WIP
Parts:
- J1: now left out of the parts list
Changed lines of the file:
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@@
 		(body_style 1)
 		(exclude_from_sim yes)
-		(in_bom yes)
+		(in_bom no)
 		(on_board yes)
 		(in_pos_files yes)
