File: Onboard DSP Board HW/String Preamp Test Board/_restore_backup_2026-09-08T22-06-20-533/String Preamp Test Board.kicad_pcb (KiCad board)
At the start: 2 copper layers, 85.9 x 24.5 mm, 51 parts, among them J1 Conn_01x07_Socket, J2 Conn_01x07_Socket, J3 Battery, J4 Output Jack, U1 TLV9004, U2 TLV9001IDCK, U3 TLV9001IDCK, U5 TP4054

Commit message: WIP
Parts:
- removed RV3: ~, Potentiometer_THT:Potentiometer_Alps_RK097_Single_Horizontal_Switch
- moved R26 12.4 mm to (148.1, 67.8), turned to 180 degrees
- moved C12 10.9 mm to (148.2, 65.7), turned to 0 degrees
- moved C15 10.8 mm to (140.6, 70.3), turned to 0 degrees
- moved U5 6.73 mm to (143.4, 66.5), turned to 180 degrees
- moved C7 2.31 mm to (135.1, 70.6)
- moved J4 0.90 mm to (131.2, 76.9)
Connections:
- U1 pad 10: Net-(U1C-+) -> GND
- U1 pad 11: /v+ -> (no net)
- U1 pad 4: GND -> (no net)
Routing:
- net /v+: track 114.1 -> 79.5 mm, vias 4 -> 3
- net /out: track 17.1 -> 0.00 mm
- net GND: track 16.9 -> 0.00 mm, vias 18 -> 5
- net /bat+: track 21.3 -> 7.13 mm
- net /RV3_in: track 14.0 -> 0.00 mm
- net Net-(J4-Pin_2): track 21.4 -> 15.8 mm
- net Net-(U1C-+): track 7.96 -> 2.45 mm
- net Net-(C7-Pad1): track 15.3 -> 12.9 mm
- net /p2_out: track 11.1 -> 8.73 mm
- net /buf_in: track 60.4 -> 58.5 mm
- net Net-(U1D-+): track 21.8 -> 20.6 mm
- net Net-(C2-Pad2): track 10.4 -> 9.53 mm
- net /sum_in: track 21.4 -> 22.1 mm
- net /sum_out: track 12.7 -> 12.1 mm
