File: Onboard DSP Board HW/String Preamp Test Board/_restore_backup_2026-09-08T22-06-20-533/String Preamp Test Board.kicad_sch (KiCad schematic)
At the start: 32 parts, among them J3 Battery, J4 Output Jack, U1 TLV9004, U5 TP4054

Commit message: WIP
Parts:
- removed unit 5 of U1
- added unit 5 of U1
- RV3: footprint Potentiometer_THT:Potentiometer_Alps_RK097_Single_Horizontal_Switch -> Potentiometer_THT:Potentiometer_Chinese_Single_Horizontal_Switch
Connections:
- net GND: now also U1.10 (V-)
- net v+: now also U1.3 (V+)
Changed lines of the file:
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@@
 		(unit 2)
 		(body_style 1)
-		(exclude_from_sim yes)
+		(exclude_from_sim no)
 		(in_bom no)
 		(on_board yes)
@@
 			)
 		)
-		(property "Footprint" "Potentiometer_THT:Potentiometer_Alps_RK097_Single_Horizontal_Switch"
+		(property "Footprint" "Potentiometer_THT:Potentiometer_Chinese_Single_Horizontal_Switch"
 			(at 109.22 46.99 0)
 			(hide yes)
@@
 			)
 		)
-		(property "Footprint" "Potentiometer_THT:Potentiometer_Alps_RK097_Single_Horizontal_Switch"
+		(property "Footprint" "Potentiometer_THT:Potentiometer_Chinese_Single_Horizontal_Switch"
 			(at 261.62 114.3 0)
 			(hide yes)
@@
 	)
 	(symbol
+		(lib_id "Amplifier_Operational:TLV9004xRUCR")
+		(at 176.53 64.77 0)
+		(unit 5)
+		(body_style 1)
+		(exclude_from_sim no)
+		(in_bom yes)
+		(on_board yes)
+		(in_pos_files yes)
+		(dnp no)
+		(fields_autoplaced yes)
+		(property "Reference" "U1"
+			(at 175.26 63.4999 0)
+			(show_name no)
+			(do_not_autoplace no)
+			(effects
+				(font
+					(size 1.27 1.27)
+				)
+				(justify left)
+			)
+		)
+		(property "Value" "TLV9004"
+			(at 175.26 66.0399 0)
+			(show_name no)
+			(do_not_autoplace no)
+			(effects
+				(font
+					(size 1.27 1.27)
+				)
+				(justify left)
+			)
+		)
+		(property "Footprint" "Package_SO:TSSOP-14_4.4x3.6mm_P0.4mm"
+			(at 176.53 64.77 0)
+			(hide yes)
+			(show_name no)
+			(do_not_autoplace no)
+			(effects
+				(font
+					(size 1.27 1.27)
+				)
+			)
+		)
+		(property "Datasheet" "http://www.ti.com/lit/ds/symlink/tlv9004.pdf"
+			(at 177.8 59.69 0)
+			(hide yes)
+			(show_name no)
+			(do_not_autoplace no)
+			(effects
+				(font
+					(size 1.27 1.27)
+				)
+			)
+		)
+		(property "Description" "Low-Power, Quad-Operational Amplifiers, Texas S-PX2QFN-14"
+			(at 176.53 64.77 0)
+			(hide yes)
+			(show_name no)
+			(do_not_autoplace no)
+			(effects
+				(font
+					(size 1.27 1.27)
+				)
+			)
+		)
+		(pin "3"
+		)
+		(pin "13"
+		)
+		(pin "12"
+		)
+		(pin "11"
+		)
+		(pin "8"
+		)
+		(pin "9"
+		)
+		(pin "10"
+		)
+		(pin "14"
+		)
+		(pin "4"
+		)
+		(pin "5"
+		)
+		(pin "6"
+		)
+		(pin "7"
+		)
+		(pin "1"
+		)
+		(pin "2"
+		)
+		(instances
+			(project "String Preamp Test Board"
+				(path "/17071b06-4887-4c2e-9588-4148705cb0ef"
+					(reference "U1")
+					(unit 5)
+				)
+			)
+		)
+	)
+	(symbol
 		(lib_id "Battery_Management:MCP73811T-420I-OT")
 		(at 142.24 31.75 0)
@@
 				)
 			)
-		)
-	)
-	(symbol
-		(lib_id "Amplifier_Operational:Opamp_Quad")
-		(at 176.53 64.77 0)
-		(mirror x)
-		(unit 5)
-		(body_style 1)
-		(exclude_from_sim no)
-		(in_bom yes)
-		(on_board yes)
-		(in_pos_files yes)
-		(dnp no)
-		(property "Reference" "U1"
-			(at 178.054 59.944 0)
-			(show_name no)
-			(do_not_autoplace no)
-			(effects
-				(font
-					(size 1.27 1.27)
-				)
-			)
-		)
-		(property "Value" "TLV9004"
-			(at 179.832 70.104 0)
-			(show_name no)
-			(do_not_autoplace no)
-			(effects
-				(font
-					(size 1.27 1.27)
-				)
-			)
-		)
-		(property "Footprint" "Package_SO:TSSOP-14_4.4x3.6mm_P0.4mm"
-			(at 176.53 64.77 0)
-			(hide yes)
-			(show_name no)
-			(do_not_autoplace no)
-			(effects
-				(font
-					(size 1.27 1.27)
-				)
-			)
-		)
-		(property "Datasheet" ""
-			(at 176.53 64.77 0)
-			(hide yes)
-			(show_name no)
-			(do_not_autoplace no)
-			(effects
-				(font
-					(size 1.27 1.27)
-				)
-			)
-		)
-		(property "Description" "Quad operational amplifier"
-			(at 176.53 55.88 0)
-			(hide yes)
-			(show_name no)
-			(do_not_autoplace no)
-			(effects
-				(font
-					(size 1.27 1.27)
-				)
-			)
-		)
-		(property "Sim.Library" "tlv9004.lib"
-			(at 163.83 52.07 0)
-			(hide yes)
-			(show_name yes)
-			(do_not_autoplace no)
-			(effects
-				(font
-					(size 1.27 1.27)
-				)
-				(justify left)
-			)
-		)
-		(property "Sim.Name" "TLV9004"
-			(at 163.83 44.45 0)
-			(hide yes)
-			(show_name yes)
-			(do_not_autoplace no)
-			(effects
-				(font
-					(size 1.27 1.27)
-				)
-				(justify left)
-			)
-		)
-		(property "Sim.Device" "SUBCKT"
-			(at 163.83 46.99 0)
-			(hide yes)
-			(show_name yes)
-			(do_not_autoplace no)
-			(effects
-				(font
-					(size 1.27 1.27)
-				)
-				(justify left)
-			)
-		)
-		(property "Sim.Pins" "1=OUT1 2=IN1- 3=IN1+ 4=VCC 5=IN2+ 6=IN2- 7=OUT2 8=OUT3 9=IN3- 10=IN3+ 11=VEE 12=IN4+ 13=IN4- 14=OUT4"
-			(at 163.83 49.53 0)
-			(hide yes)
-			(show_name yes)
-			(do_not_autoplace no)
-			(effects
-				(font
-					(size 1.27 1.27)
-				)
-				(justify left)
-			)
-		)
-		(property private "KLC_S3.1" "Units A+B are centered, UnitC has a offset so it fits nicely on A or B."
-			(at 163.83 40.64 0)
-			(hide yes)
-			(show_name yes)
-			(do_not_autoplace no)
-			(effects
-				(font
-					(size 1.27 1.27)
-				)
-				(justify left)
-			)
-		)
-		(property private "KLC_S4.1" "Pin1 and Pin7 are the output, adding a name would look ugly and does not add a benefit."
-			(at 163.83 38.1 0)
-			(hide yes)
-			(show_name yes)
-			(do_not_autoplace no)
-			(effects
-				(font
-					(size 1.27 1.27)
-				)
-				(justify left)
-			)
-		)
-		(property private "KLC_S6.2" "This is a generic symbol and thus has no datasheet."
-			(at 163.83 35.56 0)
-			(hide yes)
-			(show_name yes)
-			(do_not_autoplace no)
-			(effects
-				(font
-					(size 1.27 1.27)
-				)
-				(justify left)
-			)
-		)
-		(pin "6"
-		)
-		(pin "14"
-		)
-		(pin "8"
-		)
-		(pin "9"
-		)
-		(pin "5"
-		)
-		(pin "12"
-		)
-		(pin "2"
-		)
-		(pin "1"
-		)
-		(pin "4"
-		)
-		(pin "11"
-		)
-		(pin "3"
-		)
-		(pin "7"
-		)
-		(pin "10"
-		)
-		(pin "13"
-		)
-		(instances
-			(project "String Preamp Test Board"
-				(path "/17071b06-4887-4c2e-9588-4148705cb0ef"
-					(reference "U1")
-					(unit 5)
-				)
-			)
